File: kicad/supply.kicad_sch (KiCad schematic)
At the start: 0 parts

Commit message: init
Parts:
- added C1, C2, C3, C4, C5: C, symbol Device:C
- added P1: USB_C_Plug_USB2.0, symbol Connector:USB_C_Plug_USB2.0
- added R1, R2, R3, R4, R5: R, symbol Device:R
- added U1: MCP73831-2-OT, Package_TO_SOT_SMD:SOT-23-5, symbol Battery_Management:MCP73831-2-OT
- added U2: ME6211C33M5, Package_TO_SOT_SMD:SOT-23-5, symbol Regulator_Linear:ME6211C33M5
Connections:
- new net: P1.A4 (VBUS), P1.A9 (VBUS), P1.B4 (VBUS), P1.B9 (VBUS)
- new net GND: P1.A1 (GND), P1.A12 (GND), P1.B1 (GND), P1.B12 (GND)

Commit message: init
Parts:
- added D1, D2: D, symbol Device:D
- added D3: LED, symbol Device:LED
- added J1: Conn_01x02_Pin, symbol Connector:Conn_01x02_Pin
- added U4: BCM857BS, libs:SOT363, symbol esp32-clock:BCM857BS
Connections:
- net GND: now also C1.2, P1.S1 (SHIELD), R2.1, R4.2, R5.2, U1.2 (V_{SS}), J1.2 (Pin_2)
- net at U1.1 (STAT): now also D3.1 (K)
- net at U1.3 (V_{BAT}): now also C1.1, J1.1 (Pin_1)
- net at U1.4 (V_{DD}): now also R3.1, D1.1 (K), U4.4 (E2)
- net at U1.5 (PROG): now also R2.2
- net at R3.2: now also D3.2 (A)
- net at R5.1: now also U4.2 (B1), U4.5 (B2), U4.6 (C1)
- net at R4.1: now also D2.1 (K), U4.3 (C2)
- new net: D1.2 (A), D2.2 (A), U4.1 (E1)
Other:
- moved on the sheet: C1, R2, R3, R4, R5, U1, U2

Commit message: init
Parts:
- removed C3: C, symbol Device:C
- removed D1, D2: D, symbol Device:D
- added D1, D7: BAT54A, Package_TO_SOT_SMD:SOT-23, symbol Diode:BAT54A
- added D4: D, Package_TO_SOT_SMD:SOT-323_SC-70, symbol Device:D
- C1, C2, C4, C5: footprint (none) -> Capacitor_SMD:C_0201_0603Metric
- D3: footprint (none) -> LED_SMD:LED_PLCC-2_3.4x3.0mm_AK
- P1: footprint (none) -> Connector_USB:USB_C_Receptacle_GCT_USB4135-GF-A_6P_TopMnt_Horizontal
- R1, R5: value R -> 10K; footprint (none) -> Resistor_SMD:R_0201_0603Metric
- R2, R3: value R -> 2K; footprint (none) -> Resistor_SMD:R_0201_0603Metric
- R4: value R -> 47K; footprint (none) -> Resistor_SMD:R_0201_0603Metric
Connections:
- net GND: now also C2.2, C4.2, C5.2, R1.2, U2.2 (V_{SS})
- net at C2.1: now also R1.1, R3.1, U1.4 (V_{DD}), U4.4 (E2), D1.2, D4.2 (A), D7.1
- net at C1.1, J1.1 (Pin_1), U1.3 (V_{BAT}): now also D7.3
- net at U4.1 (E1): now also P1.A6 (D+), D1.3
- net +3.3V: now reaches C4.1
- net +3.3V: now also C5.1, U2.5 (V_{OUT})
- net at R4.1, U4.3 (C2): now also D1.1
- net at U2.1 (V_{IN}): now also U2.3 (CE), D4.1 (K), D7.2
Other:
- moved on the sheet: C1, C2, C4, C5, P1, R1, U2

Commit message: init
Parts:
- removed D4: D, Package_TO_SOT_SMD:SOT-323_SC-70, symbol Device:D
- added D2: 1N4148, Diode_THT:D_DO-35_SOD27_P7.62mm_Horizontal, symbol Diode:1N4148
- C1, C2: value C -> 4,7µF
- C4: value C -> 100nF
- C5: value C -> 10µF
- J1: value Conn_01x02_Pin -> Battery Connector
- R3: value 2K -> 470
- U2: value ME6211C33M5 -> ME6211
Connections:
- net at C2.1, D1.2, D7.1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: now also D2.2 (A)
- net at D7.2, U2.1 (V_{IN}), U2.3 (CE): now also D2.1 (K)

Commit message: init
Parts:
- J1: footprint (none) -> Connector:JWT_A3963_1x02_P3.96mm_Vertical
- U2: value ME6211 -> ME6211H33M5G
Changed lines of the file:
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@@
 			)
 		)
-		(property "Value" "ME6211"
+		(property "Value" "ME6211H33M5G"
 			(at 244.475 78.105 0)
 			(effects
@@
 			)
 		)
-		(property "Footprint" ""
+		(property "Footprint" "Connector:JWT_A3963_1x02_P3.96mm_Vertical"
 			(at 118.745 113.03 0)
 			(effects

Commit message: init
Connections:
- net USB_D_N: now reaches P1.A7 (D-)
Changed lines of the file:
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@@
+	(wire
+		(pts
+			(xy 85.09 78.105) (xy 77.47 78.105)
+		)
+		(stroke
+			(width 0)
+			(type default)
+		)
+	)
 	(wire
 		(pts
@@
 		)
 	)
+	(hierarchical_label "USB_D_N"
+		(shape input)
+		(at 85.09 78.105 0)
+		(fields_autoplaced yes)
+		(effects
+			(font
+				(size 1.27 1.27)
+			)
+			(justify left)
+		)
+	)

Commit message: init
Parts:
- added C7: 100nF, symbol Device:C
- added C8: 1µF, symbol Device:C
- added R7: 5.1K, Resistor_SMD:R_0201_0603Metric, symbol Device:R
- added U5: CP2102N-Axx-xQFN20, Package_DFN_QFN:SiliconLabs_QFN-20-1EP_3x3mm_P0.5mm, symbol Interface_USB:CP2102N-Axx-xQFN20
Connections:
- net +3.3V: now also P1.A4 (VBUS), P1.A9 (VBUS), P1.B4 (VBUS), P1.B9 (VBUS), C7.1, C8.1, U5.8 (VBUS)
- net GND: now also C7.2, C8.2, R7.1, U5.12 (GND), U5.21 (GND), U5.3 (GND)
- net at D1.3, P1.A6 (D+), U4.1 (E1): now also U5.4 (D+)
- net at P1.A5 (CC): now also R7.2
- net USB_D_N: no longer names the net of P1.A7 (D-)
- net USB_D_N: now also U5.5 (D-)
- new net RTS: U5.16 (~{RTS})
- new net RXD: U5.17 (RXD)
- new net TXD: U5.18 (TXD)

Commit message: init
Parts:
- added C10: 0,1µF, Capacitor_SMD:C_0201_0603Metric, symbol Device:C
- added C9: 4,7µF, Capacitor_SMD:C_0201_0603Metric, symbol Device:C
- added R8: 2K, symbol Device:R
- added R9: 10K, symbol Device:R
Connections:
- net +3.3V: now also U5.6 (VDD), U5.7 (VREGIN), C10.2, C9.2, R8.2
- net GND: now also C10.1, C9.1, R9.2
- net at U5.11 (~{SUSPEND}): now also R9.1
- net RTS: no longer names the net of U5.16 (~{RTS})
- net RTS: now also R8.1
