File: kicad/supply.kicad_sch (KiCad schematic)
At the start: 26 parts, among them J1 Battery Connector, P1 USB_C_Plug_USB2.0, U1 MCP73831-2-OT, U2 ME6211H33M5G, U4 BCM857BS, U5 CP2102N-Axx-xQFN20

Commit message: init
Parts:
- C7, C8: footprint (none) -> Capacitor_SMD:C_0201_0603Metric
- R8, R9: footprint (none) -> Resistor_SMD:R_0201_0603Metric
- U5: footprint Package_DFN_QFN:SiliconLabs_QFN-20-1EP_3x3mm_P0.5mm -> Package_DFN_QFN:QFN-20-1EP_3x3mm_P0.45mm_EP1.6x1.6mm
Connections:
- net +3.3V: no longer C10.2, C7.1, C8.1, C9.2, P1.A4 (VBUS), P1.A9 (VBUS), P1.B4 (VBUS), P1.B9 (VBUS), U5.6 (VDD), U5.7 (VREGIN), U5.8 (VBUS)
- net GND: now also U2.3 (CE)
- net at D2.1 (K), D7.2, U2.1 (V_{IN}): no longer U2.3 (CE)
- new net +5V: C10.2, C7.1, C8.1, C9.2, P1.A4 (VBUS), P1.A9 (VBUS), P1.B4 (VBUS), P1.B9 (VBUS), U5.6 (VDD), U5.7 (VREGIN), U5.8 (VBUS)
Changed lines of the file:
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@@
 	)
 	(junction
-		(at 231.775 83.185)
-		(diameter 0)
-		(color 0 0 0 0)
-	)
-	(junction
 		(at 83.82 65.405)
 		(diameter 0)
@@
 	)
 	(junction
+		(at 244.475 97.155)
+		(diameter 0)
+		(color 0 0 0 0)
+	)
+	(junction
 		(at 139.065 113.03)
 		(diameter 0)
@@
 	(wire
 		(pts
+			(xy 88.265 60.96) (xy 88.265 65.405)
+		)
+		(stroke
+			(width 0)
+			(type default)
+		)
+	)
+	(wire
+		(pts
 			(xy 89.535 107.315) (xy 89.535 114.3)
 		)
@@
 	(wire
 		(pts
-			(xy 231.775 85.725) (xy 231.775 83.185)
+			(xy 234.95 85.725) (xy 234.95 97.155)
 		)
 		(stroke
@@
 	(wire
 		(pts
-			(xy 236.855 85.725) (xy 231.775 85.725)
-		)
-		(stroke
-			(width 0)
-			(type default)
-		)
-	)
-	(wire
-		(pts
 			(xy 200.025 83.185) (xy 203.835 83.185)
 		)
@@
 	(wire
 		(pts
+			(xy 236.855 85.725) (xy 234.95 85.725)
+		)
+		(stroke
+			(width 0)
+			(type default)
+		)
+	)
+	(wire
+		(pts
 			(xy 120.015 153.67) (xy 127.635 153.67)
 		)
@@
 	(wire
 		(pts
-			(xy 219.075 83.185) (xy 231.775 83.185)
-		)
-		(stroke
-			(width 0)
-			(type default)
-		)
-	)
-	(wire
-		(pts
 			(xy 81.28 142.875) (xy 81.28 78.105)
 		)
@@
 	(wire
 		(pts
-			(xy 83.82 61.595) (xy 83.82 65.405)
+			(xy 54.61 103.505) (xy 54.61 106.045)
 		)
 		(stroke
@@
 	(wire
 		(pts
-			(xy 54.61 103.505) (xy 54.61 106.045)
+			(xy 79.375 70.485) (xy 79.375 60.96)
 		)
 		(stroke
@@
 	(wire
 		(pts
-			(xy 79.375 70.485) (xy 79.375 60.96)
+			(xy 175.26 127) (xy 175.26 83.185)
 		)
 		(stroke
@@
 	(wire
 		(pts
-			(xy 175.26 127) (xy 175.26 83.185)
+			(xy 100.965 107.315) (xy 100.965 114.3)
 		)
 		(stroke
@@
 	(wire
 		(pts
-			(xy 100.965 107.315) (xy 100.965 114.3)
+			(xy 234.95 97.155) (xy 244.475 97.155)
 		)
 		(stroke
@@
 	(wire
 		(pts
-			(xy 231.775 83.185) (xy 236.855 83.185)
+			(xy 219.075 83.185) (xy 236.855 83.185)
 		)
 		(stroke
@@
 	)
 	(symbol
-		(lib_id "power:+3.3V")
-		(at 83.82 61.595 0)
-		(unit 1)
-		(exclude_from_sim no)
-		(in_bom yes)
-		(on_board yes)
-		(dnp no)
-		(fields_autoplaced yes)
-		(property "Reference" "#PWR016"
-			(at 83.82 65.405 0)
-			(effects
-				(font
-					(size 1.27 1.27)
-				)
-				(hide yes)
-			)
-		)
-		(property "Value" "+3.3V"
-			(at 83.82 57.15 0)
-			(effects
-				(font
-					(size 1.27 1.27)
-				)
-			)
-		)
-		(property "Footprint" ""
-			(at 83.82 61.595 0)
-			(effects
-				(font
-					(size 1.27 1.27)
-				)
-				(hide yes)
-			)
-		)
-		(property "Datasheet" ""
-			(at 83.82 61.595 0)
-			(effects
-				(font
-					(size 1.27 1.27)
-				)
-				(hide yes)
-			)
-		)
-		(property "Description" "Power symbol creates a global label with name \"+3.3V\""
-			(at 83.82 61.595 0)
-			(effects
-				(font
-					(size 1.27 1.27)
-				)
-				(hide yes)
-			)
-		)
-		(pin "1"
-		)
-		(instances
-			(project ""
-				(path "/705cc6fa-d5d2-496f-be92-82c69a6f5679/5f53b007-a500-4fce-b6cc-e08c4de98886"
-					(reference "#PWR016")
-					(unit 1)
-				)
-			)
-		)
-	)
-	(symbol
 		(lib_id "Device:R")
 		(at 131.445 160.02 90)
@@
 			)
 		)
-		(property "Footprint" ""
+		(property "Footprint" "Resistor_SMD:R_0201_0603Metric"
 			(at 131.445 161.798 90)
 			(effects
@@
 	)
 	(symbol
-		(lib_id "power:+3.3V")
-		(at 100.965 99.06 0)
-		(unit 1)
-		(exclude_from_sim no)
-		(in_bom yes)
-		(on_board yes)
-		(dnp no)
-		(fields_autoplaced yes)
-		(property "Reference" "#PWR019"
-			(at 100.965 102.87 0)
-			(effects
-				(font
-					(size 1.27 1.27)
-				)
-				(hide yes)
-			)
-		)
-		(property "Value" "+3.3V"
-			(at 100.965 93.98 0)
-			(effects
-				(font
-					(size 1.27 1.27)
-				)
-			)
-		)
-		(property "Footprint" ""
-			(at 100.965 99.06 0)
-			(effects
-				(font
-					(size 1.27 1.27)
-				)
-				(hide yes)
-			)
-		)
-		(property "Datasheet" ""
-			(at 100.965 99.06 0)
-			(effects
-				(font
-					(size 1.27 1.27)
-				)
-				(hide yes)
-			)
-		)
-		(property "Description" "Power symbol creates a global label with name \"+3.3V\""
-			(at 100.965 99.06 0)
-			(effects
-				(font
-					(size 1.27 1.27)
-				)
-				(hide yes)
-			)
-		)
-		(pin "1"
-		)
-		(instances
-			(project ""
-				(path "/705cc6fa-d5d2-496f-be92-82c69a6f5679/5f53b007-a500-4fce-b6cc-e08c4de98886"
-					(reference "#PWR019")
-					(unit 1)
-				)
-			)
-		)
-	)
-	(symbol
 		(lib_id "Interface_USB:CP2102N-Axx-xQFN20")
 		(at 100.965 150.495 0)
@@
 			)
 		)
-		(property "Footprint" "Package_DFN_QFN:SiliconLabs_QFN-20-1EP_3x3mm_P0.5mm"
+		(property "Footprint" "Package_DFN_QFN:QFN-20-1EP_3x3mm_P0.45mm_EP1.6x1.6mm"
 			(at 132.715 177.165 0)
 			(effects
@@
 			)
 		)
-		(property "Footprint" ""
+		(property "Footprint" "Capacitor_SMD:C_0201_0603Metric"
 			(at 96.2152 74.93 0)
 			(effects
@@
 	)
 	(symbol
+		(lib_id "power:+5V")
+		(at 100.965 99.06 0)
+		(unit 1)
+		(exclude_from_sim no)
+		(in_bom yes)
+		(on_board yes)
+		(dnp no)
+		(fields_autoplaced yes)
+		(property "Reference" "#PWR022"
+			(at 100.965 102.87 0)
+			(effects
+				(font
+					(size 1.27 1.27)
+				)
+				(hide yes)
+			)
+		)
+		(property "Value" "+5V"
+			(at 100.965 93.98 0)
+			(effects
+				(font
+					(size 1.27 1.27)
+				)
+			)
+		)
+		(property "Footprint" ""
+			(at 100.965 99.06 0)
+			(effects
+				(font
+					(size 1.27 1.27)
+				)
+				(hide yes)
+			)
+		)
+		(property "Datasheet" ""
+			(at 100.965 99.06 0)
+			(effects
+				(font
+					(size 1.27 1.27)
+				)
+				(hide yes)
+			)
+		)
+		(property "Description" "Power symbol creates a global label with name \"+5V\""
+			(at 100.965 99.06 0)
+			(effects
+				(font
+					(size 1.27 1.27)
+				)
+				(hide yes)
+			)
+		)
+		(pin "1"
+		)
+		(instances
+			(project "esp32-clock"
+				(path "/705cc6fa-d5d2-496f-be92-82c69a6f5679/5f53b007-a500-4fce-b6cc-e08c4de98886"
+					(reference "#PWR022")
+					(unit 1)
+				)
+			)
+		)
+	)
+	(symbol
 		(lib_id "Diode:BAT54A")
 		(at 111.125 73.025 270)
@@
 	)
 	(symbol
+		(lib_id "power:+5V")
+		(at 88.265 60.96 0)
+		(unit 1)
+		(exclude_from_sim no)
+		(in_bom yes)
+		(on_board yes)
+		(dnp no)
+		(fields_autoplaced yes)
+		(property "Reference" "#PWR016"
+			(at 88.265 64.77 0)
+			(effects
+				(font
+					(size 1.27 1.27)
+				)
+				(hide yes)
+			)
+		)
+		(property "Value" "+5V"
+			(at 88.265 55.88 0)
+			(effects
+				(font
+					(size 1.27 1.27)
+				)
+			)
+		)
+		(property "Footprint" ""
+			(at 88.265 60.96 0)
+			(effects
+				(font
+					(size 1.27 1.27)
+				)
+				(hide yes)
+			)
+		)
+		(property "Datasheet" ""
+			(at 88.265 60.96 0)
+			(effects
+				(font
+					(size 1.27 1.27)
+				)
+				(hide yes)
+			)
+		)
+		(property "Description" "Power symbol creates a global label with name \"+5V\""
+			(at 88.265 60.96 0)
+			(effects
+				(font
+					(size 1.27 1.27)
+				)
+				(hide yes)
+			)
+		)
+		(pin "1"
+		)
+		(instances
+			(project ""
+				(path "/705cc6fa-d5d2-496f-be92-82c69a6f5679/5f53b007-a500-4fce-b6cc-e08c4de98886"
+					(reference "#PWR016")
+					(unit 1)
+				)
+			)
+		)
+	)
+	(symbol
 		(lib_id "Device:R")
 		(at 187.96 90.805 0)
@@
 			)
 		)
-		(property "Footprint" ""
+		(property "Footprint" "Resistor_SMD:R_0201_0603Metric"
 			(at 131.445 149.733 90)
 			(effects
@@
 			)
 		)
-		(property "Footprint" ""
+		(property "Footprint" "Capacitor_SMD:C_0201_0603Metric"
 			(at 89.2302 74.93 0)
 			(effects

Commit message: init
Parts:
- C10: renamed from C5; footprint Capacitor_SMD:C_0201_0603Metric -> Capacitor_SMD:C_1206_3216Metric
- C3: renamed from C8; footprint Capacitor_SMD:C_0201_0603Metric -> Capacitor_SMD:C_1206_3216Metric
- C4: renamed from C7; footprint Capacitor_SMD:C_0201_0603Metric -> Capacitor_SMD:C_1206_3216Metric
- C5: renamed from C9; footprint Capacitor_SMD:C_0201_0603Metric -> Capacitor_SMD:C_1206_3216Metric
- C6: renamed from C10; footprint Capacitor_SMD:C_0201_0603Metric -> Capacitor_SMD:C_1206_3216Metric
- C7: renamed from C2; footprint Capacitor_SMD:C_0201_0603Metric -> Capacitor_SMD:C_1206_3216Metric
- C8: renamed from C1; footprint Capacitor_SMD:C_0201_0603Metric -> Capacitor_SMD:C_1206_3216Metric
- C9: renamed from C4; footprint Capacitor_SMD:C_0201_0603Metric -> Capacitor_SMD:C_1206_3216Metric
- D3: renamed from D2; footprint Diode_THT:D_DO-35_SOD27_P7.62mm_Horizontal -> Diode_SMD:D_SMB
- R2: renamed from R7; footprint Resistor_SMD:R_0201_0603Metric -> Resistor_SMD:R_2816_7142Metric
- R3: footprint Resistor_SMD:R_0201_0603Metric -> Resistor_SMD:R_2816_7142Metric
- R4: renamed from R8; footprint Resistor_SMD:R_0201_0603Metric -> Resistor_SMD:R_2816_7142Metric
- R5: renamed from R9; footprint Resistor_SMD:R_0201_0603Metric -> Resistor_SMD:R_2816_7142Metric
- R6: renamed from R5; footprint Resistor_SMD:R_0201_0603Metric -> Resistor_SMD:R_2816_7142Metric
- R7: renamed from R2; footprint Resistor_SMD:R_0201_0603Metric -> Resistor_SMD:R_2816_7142Metric
- R8: renamed from R4; footprint Resistor_SMD:R_0201_0603Metric -> Resistor_SMD:R_2816_7142Metric
- R9: renamed from R1; footprint Resistor_SMD:R_0201_0603Metric -> Resistor_SMD:R_2816_7142Metric
- renumbered D3 to D2, D7 to D4, U5 to U2, U1 to U3, U2 to U5
Other:
- moved on the sheet: D4

Commit message: init
Connections:
- no-connect marks 0 -> 1
Changed lines of the file:
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@@
 		(color 0 0 0 0)
+	)
+	(no_connect
+		(at 77.47 73.025)
 	)
 	(wire

Commit message: init
Parts:
- R2: footprint Resistor_SMD:R_2816_7142Metric -> Resistor_SMD:R_0805_2012Metric; LCSC (none) -> C57864
- R3: footprint Resistor_SMD:R_2816_7142Metric -> Resistor_SMD:R_1206_3216Metric; LCSC (none) -> C4502
- R4, R5, R6, R7, R8, R9: footprint Resistor_SMD:R_2816_7142Metric -> Resistor_SMD:R_1206_3216Metric
Connections:
- no-connect marks 1 -> 9
Other:
- moved on the sheet: C3, C5, C6, C7, C8, D1, D2, D3, J1, P1, R2, R3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

Commit message: init
Connections:
- net +3.3V: now also C5.2, C6.2, U2.6 (VDD), U2.7 (VREGIN)
- net +5V: no longer C5.2, C6.2, U2.6 (VDD), U2.7 (VREGIN)
Changed lines of the file:
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@@
+	)
+	(symbol
+		(lib_id "power:+3.3V")
+		(at 101.6 99.06 0)
+		(unit 1)
+		(exclude_from_sim no)
+		(in_bom yes)
+		(on_board yes)
+		(dnp no)
+		(fields_autoplaced yes)
+		(property "Reference" "#PWR011"
+			(at 101.6 102.87 0)
+			(effects
+				(font
+					(size 1.27 1.27)
+				)
+				(hide yes)
+			)
+		)
+		(property "Value" "+3.3V"
+			(at 101.6 94.615 0)
+			(effects
+				(font
+					(size 1.27 1.27)
+				)
+			)
+		)
+		(property "Footprint" ""
+			(at 101.6 99.06 0)
+			(effects
+				(font
+					(size 1.27 1.27)
+				)
+				(hide yes)
+			)
+		)
+		(property "Datasheet" ""
+			(at 101.6 99.06 0)
+			(effects
+				(font
+					(size 1.27 1.27)
+				)
+				(hide yes)
+			)
+		)
+		(property "Description" "Power symbol creates a global label with name \"+3.3V\""
+			(at 101.6 99.06 0)
+			(effects
+				(font
+					(size 1.27 1.27)
+				)
+				(hide yes)
+			)
+		)
+		(pin "1"
+		)
+		(instances
+			(project "esp32-clock"
+				(path "/705cc6fa-d5d2-496f-be92-82c69a6f5679/5f53b007-a500-4fce-b6cc-e08c4de98886"
+					(reference "#PWR011")
+					(unit 1)
+				)
+			)
+		)
 	)
 	(symbol
@@
 					(unit 1)
 				)
-			)
-		)
-	)
-	(symbol
-		(lib_id "power:+5V")
-		(at 101.6 99.06 0)
-		(unit 1)
-		(exclude_from_sim no)
-		(in_bom yes)
-		(on_board yes)
-		(dnp no)
-		(fields_autoplaced yes)
-		(property "Reference" "#PWR011"
-			(at 101.6 102.87 0)
-			(effects
-				(font
-					(size 1.27 1.27)
-				)
-				(hide yes)
-			)
-		)
-		(property "Value" "+5V"
-			(at 101.6 93.98 0)
-			(effects
-				(font
-					(size 1.27 1.27)
-				)
-			)
-		)
-		(property "Footprint" ""
-			(at 101.6 99.06 0)
-			(effects
-				(font
-					(size 1.27 1.27)
-				)
-				(hide yes)
-			)
-		)
-		(property "Datasheet" ""
-			(at 101.6 99.06 0)
-			(effects
-				(font
-					(size 1.27 1.27)
-				)
-				(hide yes)
-			)
-		)
-		(property "Description" "Power symbol creates a global label with name \"+5V\""
-			(at 101.6 99.06 0)
-			(effects
-				(font
-					(size 1.27 1.27)
-				)
-				(hide yes)
-			)
-		)
-		(pin "1"
-		)
-		(instances
-			(project "esp32-clock"
-				(path "/705cc6fa-d5d2-496f-be92-82c69a6f5679/5f53b007-a500-4fce-b6cc-e08c4de98886"
-					(reference "#PWR011")
-					(unit 1)
-				)

Commit message: init
Parts:
- removed C8: 4,7µF, Capacitor_SMD:C_1206_3216Metric, symbol Device:C
- removed D3: 1N4148, Diode_SMD:D_SMB, symbol Diode:1N4148
- removed J1: Battery Connector, Connector:JWT_A3963_1x02_P3.96mm_Vertical, symbol Connector:Conn_01x02_Pin
- added C11: 10µF, Capacitor_SMD:C_1206_3216Metric, symbol Device:C
- added D3: B5819WS, Diode_SMD:D_SOD-323F, symbol Device:D
- added D5: Green, LED_SMD:LED_PLCC-2_3.4x3.0mm_AK, symbol Device:LED
- added J2: Battery Connector, Connector:JWT_A3963_1x02_P3.96mm_Vertical, symbol Connector:Conn_01x02_Pin
- added R10: 470, Resistor_SMD:R_1206_3216Metric, symbol Device:R
- C9: value 100nF -> 1µF
- D2: value LED -> Red
- R7: value 2K -> 2K2
- U5: value ME6211H33M5G -> ME6211C12M5G-N; LCSC (none) -> C236672
Connections:
- net +5V: now also D1.3, U4.1 (E1)
- net GND: now also C11.2, J2.1 (Pin_1), R10.2; no longer U5.3 (CE)
- net at C7.1, D1.2, D4.1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: now also D3.2 (A)
- net at D2.1 (K), U3.1 (STAT): now also D5.2 (A)
- net at D4.3, U3.3 (V_{BAT}): now also C11.1, J2.2 (Pin_2)
- net at P1.A6 (D+), U2.4 (D+): no longer D1.3, U4.1 (E1)
- net at D4.2, U5.1 (V_{IN}): now also U5.3 (CE), D3.1 (K)
- new net: D5.1 (K), R10.1
Other:
- moved on the sheet: R7

Commit message: init
Parts:
- renumbered C11 to C8, D5 to D3, D3 to D4, D4 to D5, J2 to J1, R9 to R10, R10 to R7, R7 to R9

Commit message: init
Parts:
- R7: LCSC (none) -> C4502
Changed lines of the file:
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@@
+			)
+		)
+		(property "LCSC" "C4502"
+			(at 147.32 92.71 0)
+			(effects
+				(font
+					(size 1.27 1.27)
+				)
+				(hide yes)
 			)
 		)
