File: kicad/supply.kicad_sch (KiCad schematic)
At the start: 28 parts, among them J1 Battery Connector, P1 USB_C_Plug_USB2.0, U2 CP2102N-Axx-xQFN20, U3 MCP73831-2-OT, U4 BCM857BS, U5 ME6211C12M5G-N

Commit message: init
Parts:
- R2: footprint Resistor_SMD:R_0805_2012Metric -> Resistor_SMD:R_0603_1608Metric
- R3, R7, R8, R9: footprint Resistor_SMD:R_1206_3216Metric -> Resistor_SMD:R_0603_1608Metric
Changed lines of the file:
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@@
 			)
 		)
-		(property "Footprint" "Resistor_SMD:R_0805_2012Metric"
+		(property "Footprint" "Resistor_SMD:R_0603_1608Metric"
 			(at 78.232 57.15 90)
 			(effects
@@
 			)
 		)
-		(property "Footprint" "Resistor_SMD:R_1206_3216Metric"
+		(property "Footprint" "Resistor_SMD:R_0603_1608Metric"
 			(at 166.37 94.488 90)
 			(effects
@@
 			)
 		)
-		(property "Footprint" "Resistor_SMD:R_1206_3216Metric"
+		(property "Footprint" "Resistor_SMD:R_0603_1608Metric"
 			(at 127.762 90.17 90)
 			(effects
@@
 			)
 		)
-		(property "Footprint" "Resistor_SMD:R_1206_3216Metric"
+		(property "Footprint" "Resistor_SMD:R_0603_1608Metric"
 			(at 163.322 69.85 90)
 			(effects
@@
 			)
 		)
-		(property "Footprint" "Resistor_SMD:R_1206_3216Metric"
+		(property "Footprint" "Resistor_SMD:R_0603_1608Metric"
 			(at 147.32 94.488 90)
 			(effects

Commit message: init
Parts:
- J1: footprint Connector:JWT_A3963_1x02_P3.96mm_Vertical -> Connector_PinHeader_1.00mm:PinHeader_1x02_P1.00mm_Vertical
Changed lines of the file:
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@@
 			)
 		)
-		(property "Footprint" "Connector:JWT_A3963_1x02_P3.96mm_Vertical"
+		(property "Footprint" "Connector_PinHeader_1.00mm:PinHeader_1x02_P1.00mm_Vertical"
 			(at 240.03 132.08 0)
 			(effects
@@
 			(at 240.03 132.08 0)
 			(effects
+				(font
+					(size 1.27 1.27)
+				)
+				(hide yes)
+			)
+		)
+		(property "LCSC" ""
+			(at 240.03 132.08 0)
+			(effects

Commit message: init
Parts:
- added R11: 22K, Resistor_SMD:R_0603_1608Metric, symbol Device:R
- added R12: 47K5, Resistor_SMD:R_0603_1608Metric, symbol Device:R
- C10, C8: LCSC (none) -> C13585
- C3, C9: LCSC (none) -> C1848
- C4, C6: LCSC (none) -> C24497
- C5, C7: LCSC (none) -> C29823
- D1, D5: LCSC (none) -> C8591
- R10, R5, R6: LCSC (none) -> C17902
- R4: LCSC (none) -> C17944
- R8: LCSC (none) -> C25819
- R9: LCSC (none) -> C4190
- U2: LCSC (none) -> C969913
- U3: LCSC (none) -> C14879
Connections:
- net +5V: now also R11.1; no longer U2.8 (VBUS)
- net GND: now also R12.2
- new net: R11.2, R12.1, U2.8 (VBUS)

Commit message: init
Parts:
- added H1, H2, H3, H4: MountingHole, MountingHole:MountingHole_2.2mm_M2_DIN965_Pad, symbol Mechanical:MountingHole
- P1: LCSC (none) -> C456012

Commit message: init
Parts:
- R12: LCSC C23061 -> C25819
- R2: LCSC C57864 -> C23186
- R3, R7: LCSC C4502 -> C23179
- U4: LCSC (none) -> C20426291
Changed lines of the file:
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@@
 			)
 		)
-		(property "LCSC" "C57864"
+		(property "LCSC" "C23186"
 			(at 80.01 57.15 0)
 			(effects
@@
 			)
 		)
-		(property "LCSC" "C23061"
+		(property "LCSC" "C25819"
 			(at 85.725 151.1299 0)
 			(effects
@@
 			)
 		)
-		(property "LCSC" "C4502"
+		(property "LCSC" "C23179"
 			(at 129.54 90.17 0)
 			(effects
@@
 			)
 		)
+		(property "LCSC" "C20426291"
+			(at 157.48 41.91 0)
+			(effects
+				(font
+					(size 1.27 1.27)
+				)
+				(hide yes)
+			)
+		)
 		(pin "6"
 		)
@@
 			)
 		)
-		(property "LCSC" "C4502"
+		(property "LCSC" "C23179"
 			(at 147.32 92.71 0)
 			(effects

Commit message: init
Parts:
- J1: footprint Connector_PinHeader_1.00mm:PinHeader_1x02_P1.00mm_Vertical -> Connector_PinHeader_1.27mm:PinHeader_1x02_P1.27mm_Vertical
Changed lines of the file:
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@@
 			)
 		)
-		(property "Footprint" "Connector_PinHeader_1.00mm:PinHeader_1x02_P1.00mm_Vertical"
+		(property "Footprint" "Connector_PinHeader_1.27mm:PinHeader_1x02_P1.27mm_Vertical"
 			(at 240.03 132.08 0)
 			(effects

Commit message: init
Parts:
- J1: footprint Connector_PinHeader_1.27mm:PinHeader_1x02_P1.27mm_Vertical -> Connector_PinHeader_2.54mm:PinHeader_1x02_P2.54mm_Vertical
Changed lines of the file:
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@@
 			)
 		)
-		(property "Footprint" "Connector_PinHeader_1.27mm:PinHeader_1x02_P1.27mm_Vertical"
+		(property "Footprint" "Connector_PinHeader_2.54mm:PinHeader_1x02_P2.54mm_Vertical"
 			(at 240.03 132.08 0)
 			(effects

Commit message: init
Parts:
- D2, D3: footprint LED_SMD:LED_PLCC-2_3.4x3.0mm_AK -> Diode_SMD:D_0603_1608Metric
Changed lines of the file:
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@@
 			)
 		)
-		(property "Footprint" "LED_SMD:LED_PLCC-2_3.4x3.0mm_AK"
+		(property "Footprint" "Diode_SMD:D_0603_1608Metric"
 			(at 129.54 100.33 0)
 			(effects
@@
 			)
 		)
-		(property "Footprint" "LED_SMD:LED_PLCC-2_3.4x3.0mm_AK"
+		(property "Footprint" "Diode_SMD:D_0603_1608Metric"
 			(at 138.43 92.71 0)
 			(effects
