File: kicad/esp32-clock.kicad_pcb (KiCad board)
At the start: 2 copper layers, 16 parts, among them P1 USB_C_Plug_USB2.0, U1 MCP73831-2-OT, U2 ME6211C33M5, U4 BCM857BS

Commit message: init
Parts:
- added D2: 1N4148, Diode_THT:D_DO-35_SOD27_P7.62mm_Horizontal, F.Cu at (132.4, 54.0)
- added D3: LED, LED_SMD:LED_PLCC-2_3.4x3.0mm_AK, F.Cu at (147.0, 63.5)
- added J1: Battery Connector, Connector:JWT_A3963_1x02_P3.96mm_Vertical, F.Cu at (123.5, 61.7)
- C1, C2: value C -> 4,7µF
- C4: value C -> 100nF
- C5: value C -> 10µF
- R3: value 2K -> 470
- U2: value ME6211C33M5 -> ME6211H33M5G
Connections:
- C2 pad 1: Net-(D4-A) -> Net-(D2-A)
- D1 pad 2: Net-(D4-A) -> Net-(D2-A)
- D7 pad 1: Net-(D4-A) -> Net-(D2-A)
- D7 pad 2: Net-(D4-K) -> Net-(D2-K)
- R1 pad 1: Net-(D4-A) -> Net-(D2-A)
- R3 pad 1: Net-(D4-A) -> Net-(D2-A)
- U1 pad 4: Net-(D4-A) -> Net-(D2-A)
- U2 pad 1: Net-(D4-K) -> Net-(D2-K)
- U2 pad 3: Net-(D4-K) -> Net-(D2-K)
- U4 pad 4: Net-(D4-A) -> Net-(D2-A)

Commit message: init
Parts:
- added C3: 0.1µF, Capacitor_SMD:C_0201_0603Metric, F.Cu at (102.7, 80.0)
- added C6: 0.1µF, Capacitor_SMD:C_0201_0603Metric, F.Cu at (102.7, 81.7)
- added R6: 10k, Resistor_SMD:R_0201_0603Metric, F.Cu at (102.7, 83.5)
- added SW1: RESET, Button_Switch_SMD:SW_SPST_CK_KMS2xxGP, F.Cu at (71.5, 76.8)
- added SW2: BOOT, Button_Switch_SMD:SW_SPST_CK_KMS2xxGP, F.Cu at (71.8, 87.5)
- added U3: ESP-12E, RF_Module:ESP-12E, F.Cu at (91.9, 81.0)
- moved D3 77.6 mm to (77.0, 97.0)
- moved D1 67.3 mm to (85.5, 97.0)
- moved D2 58.3 mm to (99.5, 102.2), turned to -90 degrees
- moved P1 55.7 mm to (76.0, 106.5), turned to 0 degrees
- moved J1 55.2 mm to (89.6, 105.2), turned to 0 degrees
- moved U1 45.7 mm to (91.1, 97.0)
- moved U4 44.8 mm to (97.4, 96.5)

Commit message: init
Parts:
- added C10: 0,1µF, Capacitor_SMD:C_0201_0603Metric, F.Cu at (119.7, 61.8)
- added C7: 100nF, Capacitor_SMD:C_0201_0603Metric, F.Cu at (119.7, 56.5)
- added C8: 1µF, Capacitor_SMD:C_0201_0603Metric, F.Cu at (119.7, 58.2)
- added C9: 4,7µF, Capacitor_SMD:C_0201_0603Metric, F.Cu at (119.7, 60.0)
- added R7: 5.1K, Resistor_SMD:R_0201_0603Metric, F.Cu at (119.7, 63.5)
- added R8: 2K, Resistor_SMD:R_0201_0603Metric, F.Cu at (119.7, 65.2)
- added R9: 10K, Resistor_SMD:R_0201_0603Metric, F.Cu at (119.7, 67.0)
- added U5: CP2102N-Axx-xQFN20, Package_DFN_QFN:QFN-20-1EP_3x3mm_P0.45mm_EP1.6x1.6mm, F.Cu at (123.5, 58.3)
Connections:
- P1 pad A5: unconnected-(P1-CC-PadA5) -> Net-(P1-CC)
- P1 pad A9: Net-(P1-VBUS-PadA4) -> +3.3V
- P1 pad B9: Net-(P1-VBUS-PadA4) -> +3.3V
- U2 pad 3: Net-(D2-K) -> GND
- U3 pad 21: unconnected-(U3-GPIO3/RXD-Pad21) -> /supply/RXD
- U3 pad 22: unconnected-(U3-GPIO1/TXD-Pad22) -> /supply/TXD

Commit message: init
Parts:
- C1: renamed from C3; footprint Capacitor_SMD:C_0201_0603Metric -> Capacitor_SMD:C_1206_3216Metric
- C10: renamed from C5; footprint Capacitor_SMD:C_0201_0603Metric -> Capacitor_SMD:C_1206_3216Metric
- C2: renamed from C6; footprint Capacitor_SMD:C_0201_0603Metric -> Capacitor_SMD:C_1206_3216Metric
- C3: renamed from C8; footprint Capacitor_SMD:C_0201_0603Metric -> Capacitor_SMD:C_1206_3216Metric
- C4: renamed from C7; footprint Capacitor_SMD:C_0201_0603Metric -> Capacitor_SMD:C_1206_3216Metric
- C5: renamed from C9; footprint Capacitor_SMD:C_0201_0603Metric -> Capacitor_SMD:C_1206_3216Metric
- C6: renamed from C10; footprint Capacitor_SMD:C_0201_0603Metric -> Capacitor_SMD:C_1206_3216Metric
- C7: renamed from C2; footprint Capacitor_SMD:C_0201_0603Metric -> Capacitor_SMD:C_1206_3216Metric
- C8: renamed from C1; footprint Capacitor_SMD:C_0201_0603Metric -> Capacitor_SMD:C_1206_3216Metric
- C9: renamed from C4; footprint Capacitor_SMD:C_0201_0603Metric -> Capacitor_SMD:C_1206_3216Metric
- D3: renamed from D2; footprint Diode_THT:D_DO-35_SOD27_P7.62mm_Horizontal -> Diode_SMD:D_SMB
- D4: value D -> BAT54A; footprint Package_TO_SOT_SMD:SOT-323_SC-70 -> Package_TO_SOT_SMD:SOT-23
- R1: renamed from R6; footprint Resistor_SMD:R_0201_0603Metric -> Resistor_SMD:R_2816_7142Metric
- R2: renamed from R7; footprint Resistor_SMD:R_0201_0603Metric -> Resistor_SMD:R_2816_7142Metric
- R3: footprint Resistor_SMD:R_0201_0603Metric -> Resistor_SMD:R_2816_7142Metric
- R4: renamed from R8; footprint Resistor_SMD:R_0201_0603Metric -> Resistor_SMD:R_2816_7142Metric
- R5: renamed from R9; footprint Resistor_SMD:R_0201_0603Metric -> Resistor_SMD:R_2816_7142Metric
- R6: renamed from R5; footprint Resistor_SMD:R_0201_0603Metric -> Resistor_SMD:R_2816_7142Metric
- R7: renamed from R2; footprint Resistor_SMD:R_0201_0603Metric -> Resistor_SMD:R_2816_7142Metric
- R8: renamed from R4; footprint Resistor_SMD:R_0201_0603Metric -> Resistor_SMD:R_2816_7142Metric
- R9: renamed from R1; footprint Resistor_SMD:R_0201_0603Metric -> Resistor_SMD:R_2816_7142Metric
- moved R7 30.2 mm to (133.0, 107.0), turned to 180 degrees
- moved R1 29.5 mm to (119.0, 108.0)
- moved R4 17.5 mm to (137.0, 63.0)
- moved R2 16.5 mm to (103.5, 60.0)
- moved C2 16.4 mm to (115.5, 92.0)
- moved D4 15.3 mm to (126.4, 77.5)
- moved C1 14.7 mm to (117.0, 76.5)
- moved R5 14.6 mm to (134.0, 70.0)
- moved R8 12.8 mm to (165.0, 79.5)
- moved C5 12.5 mm to (110.5, 68.5)
- moved R3 11.3 mm to (151.5, 76.5)
- moved U5 11.2 mm to (124.4, 93.0)
- moved R9 11.1 mm to (162.0, 88.5)
- moved R6 10.2 mm to (159.5, 99.5)
- moved C3 9.14 mm to (117.0, 67.0)
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- renumbered D3 to D2, D7 to D4, U3 to U1, U5 to U2, U1 to U3, U2 to U5
Connections:
- C3 pad 1: +3.3V -> +5V
- C4 pad 1: +3.3V -> +5V
- C5 pad 2: +3.3V -> +5V
- C6 pad 2: +3.3V -> +5V
- C7 pad 1: Net-(D2-A) (its old number) -> Net-(D3-A)
- D1 pad 2: Net-(D2-A) (its old number) -> Net-(D3-A)
- D3 pad 1: Net-(D2-K) (its old number) -> Net-(D3-K)
- D3 pad 2: Net-(D2-A) (its old number) -> Net-(D3-A)
- D4 pad 1: Net-(D2-A) (its old number) -> Net-(D3-A)
- D4 pad 2: Net-(D2-K) (its old number) -> Net-(D3-K)
- D4 pad 1: Net-(D4-K) -> Net-(D3-A)
- D4 pad 2: Net-(D4-A) -> Net-(D3-K)
- D4 pad 3: (no net) -> Net-(J1-Pin_1)
- P1 pad A9: +3.3V -> +5V
- P1 pad B9: +3.3V -> +5V
- R3 pad 1: Net-(D2-A) (its old number) -> Net-(D3-A)
- R9 pad 1: Net-(D2-A) (its old number) -> Net-(D3-A)
- U2 pad 6: +3.3V -> +5V
- U2 pad 7: +3.3V -> +5V
- U2 pad 8: +3.3V -> +5V
- U3 pad 4: Net-(D2-A) (its old number) -> Net-(D3-A)
- U4 pad 4: Net-(D2-A) (its old number) -> Net-(D3-A)
- U5 pad 1: Net-(D2-K) (its old number) -> Net-(D3-K)

Commit message: init
Parts:
- moved D4 3.10 mm to (133.0, 88.1)
Changed lines of the file:
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@@
 		(tags "resistor")
 		(property "Reference" "R7"
-			(at 0 -3.18 360)
+			(at 0 -3.18 0)
 			(layer "F.SilkS")
 			(effects
@@
 		)
 		(property "Value" "2K"
-			(at 0 3.18 360)
+			(at 0 3.18 0)
 			(layer "F.Fab")
 			(effects
@@
 		)
 		(fp_text user "${REFERENCE}"
-			(at 0 0 360)
+			(at 0 0 0)
 			(layer "F.Fab")
 			(effects
@@
 	(footprint "Package_TO_SOT_SMD:SOT-23"
 		(layer "F.Cu")
-		(at 134 91 -90)
+		(at 133 88.0625 -90)
 		(descr "SOT, 3 Pin (JEDEC TO-236 Var AB https://www.jedec.org/document_search?search_api_views_fulltext=TO-236), generated with kicad-footprint-generator ipc_gullwing_generator.py")
 		(tags "SOT TO_SOT_SMD")

Commit message: init
Parts:
- R1, R3, R4, R5, R6, R7, R8, R9: footprint Resistor_SMD:R_2816_7142Metric -> Resistor_SMD:R_1206_3216Metric
- R2: footprint Resistor_SMD:R_2816_7142Metric -> Resistor_SMD:R_0805_2012Metric
- moved R9 92.8 mm to (70.5, 104.0)
- moved R3 84.4 mm to (69.0, 94.0)
- moved R6 82.2 mm to (81.0, 75.0)
- moved J1 78.4 mm to (167.0, 93.0)
- moved D1 78.0 mm to (159.0, 71.0)
- moved U3 77.5 mm to (166.0, 77.0)
- moved D3 70.8 mm to (166.0, 69.0)
- moved C10 70.2 mm to (81.5, 97.0)
- moved R4 69.3 mm to (87.0, 111.0)
- moved C7 67.6 mm to (77.0, 109.5)
- moved P1 61.4 mm to (111.0, 56.0)
- moved U4 61.0 mm to (160.0, 84.0)
- moved R7 57.7 mm to (82.0, 80.0)
- moved C1 50.6 mm to (67.0, 84.0)
- moved U5 48.1 mm to (171.0, 105.0)
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Other:
- board outline added: 112.5 x 64 mm

Commit message: init
Parts:
- added D3: Green, LED_SMD:LED_PLCC-2_3.4x3.0mm_AK, F.Cu at (158.5, 94.0)
- added D5: BAT54A, Package_TO_SOT_SMD:SOT-23, F.Cu at (138.7, 94.7)
- added R10: 10K, Resistor_SMD:R_1206_3216Metric, F.Cu at (144.5, 80.0)
- C8: value 4,7µF -> 10µF
- C9: value 100nF -> 1µF
- D2: value LED -> Red
- D3: value 1N4148 -> Green; footprint Diode_SMD:D_SMB -> LED_SMD:LED_PLCC-2_3.4x3.0mm_AK
- D4 (x2): value BAT54A -> B5819WS; footprint Package_TO_SOT_SMD:SOT-23 -> Diode_SMD:D_SOD-323F
- R7: value 2K -> 470
- R9: value 10K -> 2K2
- U5: value ME6211H33M5G -> ME6211C12M5G-N
- moved J1 43.5 mm to (135.3, 63.2)
- moved C8 25.8 mm to (135.0, 70.5)
Connections:
- C5 pad 2: +5V -> +3.3V
- C6 pad 2: +5V -> +3.3V
- C7 pad 1: Net-(D3-A) -> Net-(D4-A)
- C8 pad 1: Net-(J1-Pin_1) -> Net-(J1-Pin_2)
- D1 pad 2: Net-(D3-A) -> Net-(D4-A)
- D1 pad 3: Net-(P1-D+) -> +5V
- D3 pad 2: Net-(D3-A) -> Net-(D2-K)
- D4 pad 1: Net-(D3-A) -> Net-(D4-K) (x2)
- D4 pad 2: Net-(D3-K) -> Net-(D4-A) (x2)
- J1 pad 1: Net-(J1-Pin_1) -> GND
- J1 pad 2: GND -> Net-(J1-Pin_2)
- R3 pad 1: Net-(D3-A) -> Net-(D4-A)
- R7 pad 1: GND -> Net-(D3-K)
- R7 pad 2: Net-(U3-PROG) -> GND
- R9 pad 1: Net-(D3-A) -> GND
- R9 pad 2: GND -> Net-(U3-PROG)
- U2 pad 6: +5V -> +3.3V
- U2 pad 7: +5V -> +3.3V
- U3 pad 3: Net-(J1-Pin_1) -> Net-(J1-Pin_2)
- U3 pad 4: Net-(D3-A) -> Net-(D4-A)
- U4 pad 1: Net-(P1-D+) -> +5V
- U4 pad 4: Net-(D3-A) -> Net-(D4-A)
- U5 pad 1: Net-(D3-K) -> Net-(D4-K)
- U5 pad 3: GND -> Net-(D4-K)
