File: kicad/esp32-clock.kicad_pcb (KiCad board)
At the start: 2 copper layers, 112.5 x 64 mm, 36 parts, among them J1 Battery Connector, P1 USB_C_Plug_USB2.0, SW1 RESET, SW2 BOOT, U1 ESP-12E, U2 CP2102N-Axx-xQFN20, U3 MCP73831-2-OT, U4 BCM857BS, U5 ME6211C12M5G-N

Commit message: init
Parts:
- removed the D3 at (158.5, 94.0)
- removed the D3 at (166.0, 69.0)
- removed the D4 at (155.6, 111.0)
- removed the D4 at (167.1, 111.9)
- removed U4: BCM857BS, libs:SOT363
- added D3: Green, LED_SMD:LED_PLCC-2_3.4x3.0mm_AK, F.Cu at (171.0, 53.0)
- added D4: B5819WS, Diode_SMD:D_SOD-323F, F.Cu at (125.5, 85.5)
- moved R7 86.4 mm to (168.0, 72.0), turned to 0 degrees
- moved C7 81.6 mm to (146.0, 66.0)
- moved C8 80.5 mm to (66.0, 112.0)
- moved R9 78.1 mm to (146.0, 84.0)
- moved C9 77.9 mm to (84.0, 53.0)
- moved R5 76.2 mm to (78.0, 78.0)
- moved C10 75.2 mm to (156.0, 107.0)
- moved SW2 74.0 mm to (147.0, 77.0), turned to 0 degrees
- moved C1 70.7 mm to (131.0, 54.0)
- moved C6 67.5 mm to (170.0, 67.0)
- moved SW1 65.5 mm to (132.0, 59.0), turned to 0 degrees
- moved C3 57.3 mm to (156.0, 112.0)
- moved J1 56.6 mm to (96.0, 104.0)
- moved R2 56.5 mm to (123.9, 71.5)
- moved R1 55.0 mm to (116.5, 57.0)
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Routing:
- net GND: track 0.00 -> 495.2 mm, vias 0 -> 1
- net +3.3V: track 0.00 -> 251.2 mm, vias 0 -> 5
- net Net-(D4-A): track 0.00 -> 147.2 mm, vias 0 -> 4
- net +5V: track 0.00 -> 139.3 mm, vias 0 -> 4
- net Net-(U1-GPIO0): track 0.00 -> 109.2 mm, vias 0 -> 2
- net Net-(J1-Pin_2): track 0.00 -> 94.2 mm, vias 0 -> 2
- net Net-(D2-A): track 0.00 -> 80.5 mm, vias 0 -> 2
- net Net-(D2-K): track 0.00 -> 71.9 mm, vias 0 -> 4
- net Net-(U1-EN): track 0.00 -> 68.9 mm
- net Net-(P1-CC): track 0.00 -> 37.1 mm, vias 0 -> 2
- net Net-(U2-~{RTS}): track 0.00 -> 36.5 mm, vias 0 -> 2
- net /supply/TXD: track 0.00 -> 36.5 mm, vias 0 -> 2
- net Net-(U2-~{SUSPEND}): track 0.00 -> 31.5 mm, vias 0 -> 2
- net Net-(D4-K): track 0.00 -> 30.7 mm, vias 0 -> 3
- net Net-(D3-K): track 0.00 -> 24.6 mm, vias 0 -> 2
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
Commit message: init
Parts:
- added U4: BCM857BS, libs:SOT363, F.Cu at (164.1, 98.2)
- R2: footprint Resistor_SMD:R_0805_2012Metric -> Resistor_SMD:R_0603_1608Metric
- R3, R7, R8, R9: footprint Resistor_SMD:R_1206_3216Metric -> Resistor_SMD:R_0603_1608Metric
Routing:
- net GND: track 495.2 -> 0.00 mm, vias 1 -> 0
- net +3.3V: track 251.2 -> 0.00 mm, vias 5 -> 0
- net Net-(D4-A): track 147.2 -> 0.00 mm, vias 4 -> 0
- net +5V: track 139.3 -> 0.00 mm, vias 4 -> 0
- net Net-(U1-GPIO0): track 109.2 -> 0.00 mm, vias 2 -> 0
- net Net-(J1-Pin_2): track 94.2 -> 0.00 mm, vias 2 -> 0
- net Net-(D2-A): track 80.5 -> 0.00 mm, vias 2 -> 0
- net Net-(D2-K): track 71.9 -> 0.00 mm, vias 4 -> 0
- net Net-(U1-EN): track 68.9 -> 0.00 mm
- net Net-(P1-CC): track 37.1 -> 0.00 mm, vias 2 -> 0
- net Net-(U2-~{RTS}): track 36.5 -> 0.00 mm, vias 2 -> 0
- net /supply/TXD: track 36.5 -> 0.00 mm, vias 2 -> 0
- net Net-(U2-~{SUSPEND}): track 31.5 -> 0.00 mm, vias 2 -> 0
- net Net-(D4-K): track 30.7 -> 0.00 mm, vias 3 -> 0
- net Net-(D3-K): track 24.6 -> 0.00 mm, vias 2 -> 0
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
Commit message: init
Parts:
- moved R7 91.1 mm to (86.2, 112.0)
- moved D3 88.2 mm to (85.5, 74.5), turned to -90 degrees
- moved SW1 85.8 mm to (84.5, 130.5), turned to -90 degrees
- moved R10 81.4 mm to (91.0, 109.0), turned to 180 degrees
- moved R2 63.7 mm to (87.8, 124.0)
- moved SW2 63.4 mm to (113.0, 130.5), turned to 90 degrees
- moved C7 62.2 mm to (85.5, 80.5), turned to 90 degrees
- moved C6 62.2 mm to (111.5, 88.0), turned to -90 degrees
- moved U4 60.9 mm to (104.8, 111.9), turned to 90 degrees
- moved C4 59.5 mm to (111.5, 112.0)
- moved C8 59.2 mm to (111.0, 73.5)
- moved R8 58.6 mm to (112.0, 108.0)
- moved C10 57.8 mm to (100.0, 92.5)
- moved C3 57.1 mm to (99.0, 108.5)
- moved C5 56.9 mm to (86.0, 105.5), turned to 90 degrees
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Other:
- board size 112.5 x 64 mm -> 32.5 x 63 mm

Commit message: init
Parts:
- J1: footprint Connector:JWT_A3963_1x02_P3.96mm_Vertical -> Connector_PinHeader_1.00mm:PinHeader_1x02_P1.00mm_Vertical
- moved SW2 1.57 mm to (111.8, 129.5)
- moved U3 1.49 mm to (109.2, 101.6)
- moved C10 1.43 mm to (99.1, 91.4)
- moved C3 1.35 mm to (97.8, 108.0)
- moved R10 1.34 mm to (90.2, 108.0)
- moved R5 1.26 mm to (100.3, 96.5)
- moved P1 1.23 mm to (97.8, 130.8)
- moved C8 1.22 mm to (110.5, 72.4)
- moved SW1 1.18 mm to (83.8, 129.5)
- moved R4 1.16 mm to (95.2, 102.9)
- moved C2 1.15 mm to (86.4, 99.1)
- moved R9 1.14 mm to (105.4, 91.4)
- moved R7 1.11 mm to (85.1, 111.8)
- moved R6 1.10 mm to (92.7, 91.4)
- moved U1 1.09 mm to (97.8, 74.9)
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
Commit message: init
Parts:
- added R11: 22K, Resistor_SMD:R_0603_1608Metric, F.Cu at (91.3, 107.5)
- added R12: 47K5, Resistor_SMD:R_0603_1608Metric, F.Cu at (93.0, 112.3)
- moved R10 8.85 mm to (98.0, 112.0)
- moved U2 5.72 mm to (93.6, 118.0), turned to 180 degrees
Connections:
- U2 pad 8: +5V -> Net-(U2-VBUS)

Commit message: init
Parts:
- moved C5 11.4 mm to (85.1, 116.8), turned to 0 degrees
- moved C4 11.4 mm to (110.5, 123.2)
- moved R10 8.98 mm to (105.6, 116.8), turned to 0 degrees
- moved R8 7.51 mm to (106.2, 113.0)
- moved R2 6.35 mm to (94.0, 123.2)
- moved U4 6.35 mm to (100.3, 116.8)
- moved U5 4.02 mm to (85.1, 121.9)
- moved J1 3.59 mm to (111.8, 118.1), turned to 180 degrees
- moved R7 3.59 mm to (87.6, 109.2)
- moved SW1 3.01 mm to (86.8, 129.5)
- moved U2 1.42 mm to (92.7, 116.8)
- moved R11 1.42 mm to (90.2, 106.7)
- moved P1 1.22 mm to (99.0, 130.8)
- moved SW2 0.80 mm to (111.0, 129.5)
- moved R12 0.64 mm to (92.7, 111.8)

Commit message: init
Parts:
- moved D3 30.7 mm to (109.2, 92.7), turned to 180 degrees
- moved C7 15.9 mm to (92.7, 94.0), turned to 180 degrees
- moved D5 14.8 mm to (102.9, 92.7)
- moved C3 14.4 mm to (108.0, 118.1), turned to 90 degrees
- moved C8 14.0 mm to (111.8, 86.4), turned to 90 degrees
- moved R5 13.5 mm to (110.5, 105.4)
- moved R6 10.8 mm to (100.3, 99.1), turned to 90 degrees
- moved C6 10.2 mm to (109.2, 97.8), turned to 0 degrees
- moved R8 10.0 mm to (101.6, 121.9)
- moved C10 9.92 mm to (92.7, 99.1)
- moved U3 8.98 mm to (110.5, 110.5), turned to 90 degrees
- moved R9 8.89 mm to (105.4, 100.3), turned to -90 degrees
- moved C9 6.48 mm to (110.5, 101.6), turned to 0 degrees
- moved R3 6.35 mm to (101.6, 111.8), turned to 90 degrees
- moved D1 5.08 mm to (96.5, 121.9)
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
Commit message: init
Parts:
- added H1: MountingHole, MountingHole:MountingHole_2.2mm_M2_DIN965_Pad, F.Cu at (110.5, 72.4)
- added H2: MountingHole, MountingHole:MountingHole_2.2mm_M2_DIN965_Pad, F.Cu at (85.1, 72.4)
- added H3: MountingHole, MountingHole:MountingHole_2.2mm_M2_DIN965_Pad, F.Cu at (85.1, 129.5)
- added H4: MountingHole, MountingHole:MountingHole_2.2mm_M2_DIN965_Pad, F.Cu at (110.5, 129.5)
- moved C8 17.6 mm to (95.2, 92.5), turned to -90 degrees
- moved C1 14.9 mm to (99.1, 92.9), turned to 90 degrees
- moved R3 11.6 mm to (91.4, 117.3)
- moved U2 11.3 mm to (95.4, 106.3), turned to 0 degrees
- moved R1 9.17 mm to (84.9, 104.1)
- moved R6 8.89 mm to (91.4, 99.1)
- moved D5 8.75 mm to (96.9, 99.1), turned to 0 degrees
- moved R11 8.42 mm to (96.5, 112.2), turned to 90 degrees
- moved R4 7.98 mm to (91.6, 111.8), turned to 0 degrees
- moved R5 7.92 mm to (102.7, 104.1)
- moved SW2 6.86 mm to (109.7, 122.7), turned to 0 degrees
- moved SW1 6.84 mm to (85.9, 122.7), turned to 0 degrees
- moved R12 6.63 mm to (87.6, 107.5)
- moved U5 5.44 mm to (85.4, 116.7)
- moved C4 5.28 mm to (102.7, 123.2)
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Connections:
- SW2 pad 2: unconnected-(SW2-Pad2) -> GND
Other:
- board size 32.5 x 63 mm -> 33 x 64.8 mm
