File: kicad/esp32-clock.kicad_pcb (KiCad board)
At the start: 2 copper layers, 37 x 40 mm, 34 parts, among them J1 Conn_01x07_Socket, P1 USB_C_Plug_USB2.0, Q1 BCW66G, Q2 BCW66G, SW1 RESET, SW2 BOOT, U1 ESP32-PICO-V3, U2 USBLC6-2P6, U3 AMS1117-3.3, U4 CP2102N-Axx-xQFN28

Commit message: init
Routing:
- net GND: track 177.1 -> 185.4 mm, vias 1 -> 3
- net Net-(C2-Pad1): track 61.9 -> 64.4 mm
- net Net-(Q2-B): track 45.7 -> 47.9 mm
- net /supply/TXD: track 30.5 -> 31.2 mm
Changed lines of the file:
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@@
 	)
 	(segment
+		(start 136 72.5)
+		(end 137 73.5)
+		(width 0.2)
+		(layer "F.Cu")
+		(net 1)
+	)
+	(segment
 		(start 123.3581 65.7686)
 		(end 124.1017 65.025)
@@
 	)
 	(segment
+		(start 137 73.5)
+		(end 137.7125 73.5)
+		(width 0.2)
+		(layer "F.Cu")
+		(net 1)
+	)
+	(segment
 		(start 123.358 66.1403)
 		(end 123.358 65.7686)
@@
 	)
 	(via
+		(at 136 72.5)
+		(size 0.6)
+		(drill 0.3)
+		(layers "F.Cu" "B.Cu")
+		(net 1)
+	)
+	(via
+		(at 130.5625 70.75)
+		(size 0.6)
+		(drill 0.3)
+		(layers "F.Cu" "B.Cu")
+		(net 1)
+	)
+	(via
 		(at 140.112 83.6782)
 		(size 0.6)
@@
 	)
 	(segment
+		(start 130.5625 70.75)
+		(end 134.25 70.75)
+		(width 0.2)
+		(layer "B.Cu")
+		(net 1)
+	)
+	(segment
+		(start 134.25 70.75)
+		(end 136 72.5)
+		(width 0.2)
+		(layer "B.Cu")
+		(net 1)
+	)
+	(segment
 		(start 141.1138 84.68)
 		(end 140.112 83.6782)
@@
 	)
 	(segment
-		(start 144.0066 62.7021)
-		(end 133.0191 73.6896)
-		(width 0.2)
-		(layer "B.Cu")
-		(net 16)
-	)
-	(segment
 		(start 123.6031 78.6198)
 		(end 123.2416 78.2583)
@@
 	)
 	(segment
-		(start 129.3475 73.6896)
-		(end 128.9458 74.0913)
-		(width 0.2)
-		(layer "B.Cu")
-		(net 16)
-	)
-	(segment
 		(start 127.6007 78.6198)
 		(end 123.6031 78.6198)
@@
 	)
 	(segment
-		(start 133.0191 73.6896)
+		(start 129.3475 73.6896)
+		(end 128.9458 74.0913)
+		(width 0.2)
+		(layer "B.Cu")
+		(net 16)
+	)
+	(segment
+		(start 144.0066 66.4934)
+		(end 136.8104 73.6896)
+		(width 0.2)
+		(layer "B.Cu")
+		(net 16)
+	)
+	(segment
+		(start 144.0066 62.7021)
+		(end 144.0066 66.4934)
+		(width 0.2)
+		(layer "B.Cu")
+		(net 16)
+	)
+	(segment
+		(start 136.8104 73.6896)
 		(end 129.3475 73.6896)
 		(width 0.2)
@@
 	)
 	(segment
+		(start 135.189557 68.7197)
+		(end 135.687443 68.7197)
+		(width 0.2)
+		(layer "F.Cu")
+		(net 27)
+	)
+	(segment
+		(start 135 68.909257)
+		(end 135.189557 68.7197)
+		(width 0.2)
+		(layer "F.Cu")
+		(net 27)
+	)
+	(segment
+		(start 134.3625 67.1911)
+		(end 135 67.8286)
+		(width 0.2)
+		(layer "F.Cu")
+		(net 27)
+	)
+	(segment
+		(start 135 76.3717)
+		(end 134.8239 76.5478)
+		(width 0.2)
+		(layer "F.Cu")
+		(net 27)
+	)
+	(segment
 		(start 131.3125 66.3214)
 		(end 131.3095 66.3184)
@@
 	)
 	(segment
-		(start 136.2078 75.1639)
-		(end 134.8239 76.5478)
+		(start 136.2071 71.3718)
+		(end 135 72.5789)
 		(width 0.2)
 		(layer "F.Cu")
@@
 	)
 	(segment
-		(start 134.3625 67.1911)
-		(end 136.2078 69.0364)
+		(start 136.0395 69.071757)
+		(end 136.0395 69.5398)
 		(width 0.2)
 		(layer "F.Cu")
@@
 	)
 	(segment
-		(start 134.8239 76.9227)
-		(end 134.1946 77.552)
+		(start 135 72.5789)
+		(end 135 76.3717)
+		(width 0.2)
+		(layer "F.Cu")
+		(net 27)
+	)
+	(segment
+		(start 135 67.8286)
+		(end 135 68.909257)
+		(width 0.2)
+		(layer "F.Cu")
+		(net 27)
+	)
+	(segment
+		(start 136.2071 69.7074)
+		(end 136.2071 71.3718)
 		(width 0.2)
 		(layer "F.Cu")
@@
 	)
 	(segment
-		(start 140.1237 81.1277)
-		(end 141 80.2514)
+		(start 134.8239 76.5478)
+		(end 134.8239 76.9227)
 		(width 0.2)
 		(layer "F.Cu")
@@
 	)
 	(segment
-		(start 136.2078 69.0364)
-		(end 136.2078 75.1639)
+		(start 140.1237 81.1277)
+		(end 141 80.2514)
 		(width 0.2)
 		(layer "F.Cu")
@@
 	)
 	(segment
-		(start 134.8239 76.5478)
-		(end 134.8239 76.9227)
+		(start 134.8239 76.9227)
+		(end 134.1946 77.552)
+		(width 0.2)
+		(layer "F.Cu")
+		(net 27)
+	)
+	(segment
+		(start 136.0395 69.5398)
+		(end 136.2071 69.7074)
+		(width 0.2)
+		(layer "F.Cu")
+		(net 27)
+	)
+	(segment
+		(start 135.687443 68.7197)
+		(end 136.0395 69.071757)
 		(width 0.2)
 		(layer "F.Cu")
@@
 	)
 	(segment
+		(start 134.9635 67.440043)
+		(end 134.611443 67.7921)
+		(width 0.2)
+		(layer "B.Cu")
+		(net 45)
+	)
+	(segment
 		(start 136.2755 65.2506)
-		(end 136.2755 66.129)
+		(end 134.2494 65.2506)
 		(width 0.2)
 		(layer "B.Cu")
@@
 	)
 	(segment
-		(start 130.2123 72.1922)
+		(start 133.863 65.637)
+		(end 134.004 65.778)
+		(width 0.2)
+		(layer "B.Cu")
+		(net 45)
+	)
+	(segment
+		(start 134.6389 66.617557)
+		(end 134.9635 66.942157)
+		(width 0.2)
+		(layer "B.Cu")
+		(net 45)
+	)
+	(segment
+		(start 134.2494 65.2506)
+		(end 133.863 65.637)
+		(width 0.2)
+		(layer "B.Cu")
+		(net 45)
+	)
+	(segment
+		(start 134.9635 66.942157)
+		(end 134.9635 67.440043)
+		(width 0.2)
+		(layer "B.Cu")
+		(net 45)
+	)
+	(segment
+		(start 134.6389 66.130057)
+		(end 134.6389 66.617557)
+		(width 0.2)
+		(layer "B.Cu")
+		(net 45)
+	)
+	(segment
+		(start 134.286843 65.778)
+		(end 134.6389 66.130057)
+		(width 0.2)
+		(layer "B.Cu")
+		(net 45)
+	)
+	(segment
+		(start 131.962 67.538)
+		(end 127.3078 72.1922)
+		(width 0.2)
+		(layer "B.Cu")
+		(net 45)
+	)
+	(segment
+		(start 133.913557 67.5921)
+		(end 132.0161 67.5921)
+		(width 0.2)
+		(layer "B.Cu")
+		(net 45)
+	)
+	(segment
+		(start 134.611443 67.7921)
+		(end 134.113557 67.7921)
+		(width 0.2)
+		(layer "B.Cu")
+		(net 45)
+	)
+	(segment
+		(start 132.0161 67.5921)
+		(end 131.962 67.538)
+		(width 0.2)
+		(layer "B.Cu")
+		(net 45)
+	)
+	(segment
+		(start 127.3078 72.1922)
 		(end 119.711 72.1922)
 		(width 0.2)
@@
 	)
 	(segment
-		(start 136.2755 66.129)
-		(end 130.2123 72.1922)
+		(start 134.004 65.778)
+		(end 134.286843 65.778)
+		(width 0.2)
+		(layer "B.Cu")
+		(net 45)
+	)
+	(segment
+		(start 134.113557 67.7921)
+		(end 133.913557 67.5921)
 		(width 0.2)
 		(layer "B.Cu")

Commit message: init
Parts:
- removed C8: 100nF, Capacitor_SMD:C_1206_3216Metric
- removed C9: 10µF, Capacitor_SMD:C_1206_3216Metric
- added R10: 2K, Resistor_SMD:R_1206_3216Metric, F.Cu at (143.5, 72.0)
- added R11: 2 K, Resistor_SMD:R_1206_3216Metric, F.Cu at (137.5, 93.0)
- added R12: 10 K, Resistor_SMD:R_1206_3216Metric, F.Cu at (141.5, 91.5)
- added R9: 100 K, Resistor_SMD:R_1206_3216Metric, F.Cu at (144.5, 68.0)
- R8: value 1K -> 47 K
- U1: footprint Package_DFN_QFN:QFN-48-1EP_7x7mm_P0.5mm_EP5.15x5.15mm -> Package_DFN_QFN:QFN-48-1EP_7x7mm_P0.5mm_EP5.3x5.3mm
- moved D3 0.87 mm to (149.0, 71.5)
- moved TP1 0.50 mm to (132.5, 93.0)
Connections:
- C6 pad 1: +5V -> +3.3V
- C7 pad 1: +5V -> +3.3V
- R8 pad 2: Net-(D3-A) -> Net-(U4-VBUS)
- U1 pad 25: (no net) -> unconnected-(U1-IO16-Pad25)
- U1 pad 27: Net-(J1-Pin_2) -> unconnected-(U1-IO17-Pad27)
- U1 pad 29: Net-(J1-Pin_5) -> unconnected-(U1-SD3/IO10-Pad29)
- U1 pad 34: unconnected-(U1-GPIO5-Pad34) -> Net-(J1-Pin_2)
- U1 pad 35: (no net) -> Net-(J1-Pin_5)
- U1 pad 36: (no net) -> Net-(J1-Pin_4)
- U1 pad 38: Net-(J1-Pin_1) -> unconnected-(U1-IO19-Pad38)
- U1 pad 39: Net-(J1-Pin_4) -> Net-(J1-Pin_1)
- U1 pad 44: (no net) -> unconnected-(U1-XTAL_N_NC-Pad44)
- U1 pad 45: (no net) -> unconnected-(U1-XTAL_P_NC-Pad45)
- U1 pad 47: (no net) -> unconnected-(U1-CAP2_NC-Pad47)
- U1 pad 48: (no net) -> unconnected-(U1-CAP1_NC-Pad48)
- U4 pad 11: unconnected-(U4-~{SUSPEND}-Pad11) -> Net-(U4-~{SUSPEND})
- U4 pad 8: +5V -> Net-(U4-VBUS)
- U4 pad 9: unconnected-(U4-~{RST}-Pad9) -> Net-(U4-~{RST})
Routing:
- net Net-(U4-VBUS): track 0.00 -> 41.7 mm
- net Net-(D3-A): track 47.2 -> 5.79 mm, vias 2 -> 0
- net Net-(C2-Pad1): track 64.4 -> 45.2 mm, vias 2 -> 0
- net GND: track 185.4 -> 203.5 mm, vias 3 -> 5
- net /supply/TXD: track 31.2 -> 13.7 mm, vias 4 -> 2
- net Net-(U4-~{SUSPEND}): track 0.00 -> 16.5 mm, vias 0 -> 2
- net +5V: track 59.9 -> 73.0 mm
- net +3.3V: track 135.2 -> 147.3 mm, vias 6 -> 5
- net Net-(Q2-B): track 47.9 -> 37.9 mm
- net /supply/RXD: track 39.9 -> 49.8 mm, vias 4 -> 3
- net Net-(P1-D+): track 28.4 -> 20.1 mm
- net Net-(J1-Pin_3): track 23.9 -> 17.5 mm, vias 1 -> 0
- net Net-(Q1-B): track 25.9 -> 20.7 mm
- net Net-(U1-IO12): track 27.9 -> 22.7 mm
- net Net-(U4-~{RST}): track 0.00 -> 5.14 mm
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- removed copper zone on F.Cu, net GND

Commit message: init
Connections:
- U1 pad 40: /supply/RXD -> /supply/TXD
- U1 pad 41: /supply/TXD -> /supply/RXD
Routing:
- net GND: track 203.5 -> 0.00 mm, vias 5 -> 0
- net +3.3V: track 147.3 -> 0.00 mm, vias 5 -> 0
- net +5V: track 73.0 -> 0.00 mm, vias 3 -> 0
- net /EN: track 54.1 -> 0.00 mm, vias 3 -> 0
- net /supply/RXD: track 49.8 -> 0.00 mm, vias 3 -> 0
- net Net-(C2-Pad1): track 45.2 -> 0.00 mm
- net Net-(U4-VBUS): track 41.7 -> 0.00 mm
- net /IO0: track 40.2 -> 0.00 mm, vias 2 -> 0
- net Net-(Q2-B): track 37.9 -> 0.00 mm, vias 2 -> 0
- net /RTS: track 29.3 -> 0.00 mm, vias 3 -> 0
- net Net-(D2-A): track 27.4 -> 0.00 mm
- net Net-(P1-D-): track 24.1 -> 0.00 mm, vias 2 -> 0
- net Net-(U1-IO12): track 22.7 -> 0.00 mm, vias 2 -> 0
- net Net-(Q1-B): track 20.7 -> 0.00 mm, vias 2 -> 0
- net Net-(P1-D+): track 20.1 -> 0.00 mm, vias 2 -> 0
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
Commit message: init
Parts:
- moved R7 2.10 mm to (146.5, 64.0)
- moved D2 2.06 mm to (138.0, 68.0)
- moved C2 1.80 mm to (140.5, 64.0), turned to 0 degrees
- moved H1 1.50 mm to (152.5, 60.5)
- moved D1 1.12 mm to (138.0, 72.5)
- moved U1 0.57 mm to (130.2, 71.2)
- moved R10 0.46 mm to (143.0, 72.0)
- moved R9 0.46 mm to (144.0, 68.0)
- moved Q2 0.45 mm to (128.0, 84.0)
- moved U4 0.45 mm to (135.5, 85.0)
Changed lines of the file:
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@@
 	(footprint "Resistor_SMD:R_1206_3216Metric"
 		(layer "F.Cu")
-		(at 121.98 79.9625 -90)
+		(at 122 80 -90)
 		(descr "Resistor SMD 1206 (3216 Metric), square (rectangular) end terminal, IPC-7351 nominal, (Body size source: IPC-SM-782 page 72, https://www.pcb-3d.com/wordpress/wp-content/uploads/ipc-sm-782a_amendment_1_and_2.pdf), generated with kicad-footprint-generator")
 		(tags "resistor")
 		(property "Reference" "R4"
-			(at -1.4625 1.98 90)
+			(at 0 1.98 90)
 			(layer "F.SilkS")
 			(effects
@@
 	(footprint "Diode_SMD:D_0603_1608Metric"
 		(layer "F.Cu")
-		(at 138.5 73.5)
+		(at 138 72.5)
 		(descr "Diode SMD 0603 (1608 Metric), square (rectangular) end terminal, IPC-7351 nominal, (Body size source: http://www.tortai-tech.com/upload/download/2011102023233369053.pdf), generated with kicad-footprint-generator")
 		(tags "diode")
@@
 	(footprint "Package_DFN_QFN:QFN-28-1EP_5x5mm_P0.5mm_EP3.35x3.35mm"
 		(layer "F.Cu")
-		(at 135.5 85.45)
+		(at 135.5 85)
 		(descr "QFN, 28 Pin (http://ww1.microchip.com/downloads/en/PackagingSpec/00000049BQ.pdf#page=283), generated with kicad-footprint-generator ipc_noLead_generator.py")
 		(tags "QFN NoLead")
@@
 	(footprint "MountingHole:MountingHole_2.2mm_M2_DIN965_Pad"
 		(layer "F.Cu")
-		(at 151 60.5)
+		(at 152.5 60.5)
 		(descr "Mounting Hole 2.2mm, M2, generated by kicad-footprint-generator mountinghole.py")
 		(tags "mountinghole M2 DIN965")
@@
 		(tags "capacitor")
 		(property "Reference" "C6"
-			(at 1.5 -2 90)
+			(at 0 -2 90)
 			(layer "F.SilkS")
 			(effects
@@
 	(footprint "Package_TO_SOT_SMD:SOT-23"
 		(layer "F.Cu")
-		(at 128 84.45)
+		(at 128 84)
 		(descr "SOT, 3 Pin (JEDEC TO-236 Var AB https://www.jedec.org/document_search?search_api_views_fulltext=TO-236), generated with kicad-footprint-generator ipc_gullwing_generator.py")
 		(tags "SOT TO_SOT_SMD")
@@
 	(footprint "Resistor_SMD:R_1206_3216Metric"
 		(layer "F.Cu")
-		(at 144.4625 64.5)
+		(at 146.5 64)
 		(descr "Resistor SMD 1206 (3216 Metric), square (rectangular) end terminal, IPC-7351 nominal, (Body size source: IPC-SM-782 page 72, https://www.pcb-3d.com/wordpress/wp-content/uploads/ipc-sm-782a_amendment_1_and_2.pdf), generated with kicad-footprint-generator")
 		(tags "resistor")
 		(property "Reference" "R7"
-			(at 1.5375 -2 0)
+			(at 0 -2 0)
 			(layer "F.SilkS")
 			(effects
@@
 	(footprint "Resistor_SMD:R_1206_3216Metric"
 		(layer "F.Cu")
-		(at 143.4625 72)
+		(at 143 72)
 		(descr "Resistor SMD 1206 (3216 Metric), square (rectangular) end terminal, IPC-7351 nominal, (Body size source: IPC-SM-782 page 72, https://www.pcb-3d.com/wordpress/wp-content/uploads/ipc-sm-782a_amendment_1_and_2.pdf), generated with kicad-footprint-generator")
 		(tags "resistor")
@@
 	(footprint "Package_DFN_QFN:QFN-48-1EP_7x7mm_P0.5mm_EP5.3x5.3mm"
 		(layer "F.Cu")
-		(at 130.5625 70.75)
+		(at 130.16 71.16)
 		(descr "QFN, 48 Pin (https://www.trinamic.com/fileadmin/assets/Products/ICs_Documents/TMC2041_datasheet.pdf#page=62), generated with kicad-footprint-generator ipc_noLead_generator.py")
 		(tags "QFN NoLead")
@@
 		(tags "capacitor")
 		(property "Reference" "C3"
-			(at 1 2 0)
+			(at 0 2 0)
 			(layer "F.SilkS")
 			(effects
@@
 		(tags "resistor")
 		(property "Reference" "R6"
-			(at -1.5 2 90)
+			(at 0 2 90)
 			(layer "F.SilkS")
 			(effects
@@
 	(footprint "Resistor_SMD:R_1206_3216Metric"
 		(layer "F.Cu")
-		(at 144.4625 68)
+		(at 144 68)
 		(descr "Resistor SMD 1206 (3216 Metric), square (rectangular) end terminal, IPC-7351 nominal, (Body size source: IPC-SM-782 page 72, https://www.pcb-3d.com/wordpress/wp-content/uploads/ipc-sm-782a_amendment_1_and_2.pdf), generated with kicad-footprint-generator")
 		(tags "resistor")
@@
 		(tags "resistor")
 		(property "Reference" "R5"
-			(at 1.5 -2 90)
+			(at 0 -2 90)
 			(layer "F.SilkS")
 			(effects
@@
 	(footprint "Diode_SMD:D_0603_1608Metric"
 		(layer "F.Cu")
-		(at 138.5 70)
+		(at 138 68)
 		(descr "Diode SMD 0603 (1608 Metric), square (rectangular) end terminal, IPC-7351 nominal, (Body size source: http://www.tortai-tech.com/upload/download/2011102023233369053.pdf), generated with kicad-footprint-generator")
 		(tags "diode")
@@
 	(footprint "Capacitor_SMD:C_1206_3216Metric"
 		(layer "F.Cu")
-		(at 139 65 -90)
+		(at 140.5 64)
 		(descr "Capacitor SMD 1206 (3216 Metric), square (rectangular) end terminal, IPC-7351 nominal, (Body size source: IPC-SM-782 page 76, https://www.pcb-3d.com/wordpress/wp-content/uploads/ipc-sm-782a_amendment_1_and_2.pdf), generated with kicad-footprint-generator")
 		(tags "capacitor")
 		(property "Reference" "C2"
-			(at -3 0 180)
+			(at 0 -2 180)
 			(layer "F.SilkS")
 			(effects
@@
 		)
 		(property "Value" "2,7pF"
-			(at 0 1.85 90)
+			(at 0 1.85 0)
 			(layer "F.Fab")
 			(effects
@@
 		)
 		(property "Datasheet" "~"
-			(at 0 0 90)
+			(at 0 0 0)
 			(layer "F.Fab")
 			(hide yes)
@@
 		)
 		(property "Description" "Unpolarized capacitor"
-			(at 0 0 90)
+			(at 0 0 0)
 			(layer "F.Fab")
 			(hide yes)
@@
 		(attr smd)
 		(fp_line
-			(start -0.711252 0.91)
-			(end 0.711252 0.91)
+			(start -0.711252 -0.91)
+			(end 0.711252 -0.91)
 			(stroke
 				(width 0.12)
@@
 		)
 		(fp_line
-			(start -0.711252 -0.91)
-			(end 0.711252 -0.91)
+			(start -0.711252 0.91)
+			(end 0.711252 0.91)
 			(stroke
 				(width 0.12)
@@
 		)
 		(fp_line
-			(start -2.3 1.15)
-			(end -2.3 -1.15)
+			(start -2.3 -1.15)
+			(end 2.3 -1.15)
 			(stroke
 				(width 0.05)
@@
 		)
 		(fp_line
-			(start 2.3 1.15)
-			(end -2.3 1.15)
+			(start -2.3 1.15)
+			(end -2.3 -1.15)
 			(stroke
 				(width 0.05)
@@
 		)
 		(fp_line
-			(start -2.3 -1.15)
-			(end 2.3 -1.15)
+			(start 2.3 -1.15)
+			(end 2.3 1.15)
 			(stroke
 				(width 0.05)
@@
 		)
 		(fp_line
-			(start 2.3 -1.15)
-			(end 2.3 1.15)
+			(start 2.3 1.15)
+			(end -2.3 1.15)
 			(stroke
 				(width 0.05)
@@
 		)
 		(fp_line
-			(start -1.6 0.8)
-			(end -1.6 -0.8)
+			(start -1.6 -0.8)
+			(end 1.6 -0.8)
 			(stroke
 				(width 0.1)
@@
 		)
 		(fp_line
-			(start 1.6 0.8)
-			(end -1.6 0.8)
+			(start -1.6 0.8)
+			(end -1.6 -0.8)
 			(stroke
 				(width 0.1)
@@
 		)
 		(fp_line
-			(start -1.6 -0.8)
-			(end 1.6 -0.8)
+			(start 1.6 -0.8)
+			(end 1.6 0.8)
 			(stroke
 				(width 0.1)
@@
 		)
 		(fp_line
-			(start 1.6 -0.8)
-			(end 1.6 0.8)
+			(start 1.6 0.8)
+			(end -1.6 0.8)
 			(stroke
 				(width 0.1)
@@
 		)
 		(fp_text user "${REFERENCE}"
-			(at 0 0 90)
+			(at 0 0 0)
 			(layer "F.Fab")
 			(effects
@@
 		)
 		(pad "1" smd roundrect
-			(at -1.475 0 270)
+			(at -1.475 0)
 			(size 1.15 1.8)
 			(layers "F.Cu" "F.Mask" "F.Paste")
@@
 		)
 		(pad "2" smd roundrect
-			(at 1.475 0 270)
+			(at 1.475 0)
 			(size 1.15 1.8)
 			(layers "F.Cu" "F.Mask" "F.Paste")
@@
 	(footprint "Resistor_SMD:R_1206_3216Metric"
 		(layer "F.Cu")
-		(at 127.0375 94.5)
+		(at 127 94.5)
 		(descr "Resistor SMD 1206 (3216 Metric), square (rectangular) end terminal, IPC-7351 nominal, (Body size source: IPC-SM-782 page 72, https://www.pcb-3d.com/wordpress/wp-content/uploads/ipc-sm-782a_amendment_1_and_2.pdf), generated with kicad-footprint-generator")
 		(tags "resistor")
@@
 		(tags "inductor handsolder")
 		(property "Reference" "L1"
-			(at -1.5 -2 0)
+			(at 0 -2 0)
 			(layer "F.SilkS")
 			(effects
@@
 	)
 	(gr_rect
-		(start 118.75 56.5)
-		(end 155.75 96.5)
+		(start 119 56.5)
+		(end 156 96.5)
 		(stroke
 			(width 0.05)

Commit message: init
Routing:
- net GND: track 0.00 -> 200.2 mm, vias 0 -> 4
- net +3.3V: track 0.00 -> 181.8 mm, vias 0 -> 6
- net Net-(U4-VBUS): track 0.00 -> 70.8 mm, vias 0 -> 3
- net +5V: track 0.00 -> 61.4 mm, vias 0 -> 4
- net /EN: track 0.00 -> 50.5 mm, vias 0 -> 4
- net Net-(C2-Pad1): track 0.00 -> 48.0 mm, vias 0 -> 4
- net Net-(Q2-B): track 0.00 -> 45.3 mm, vias 0 -> 2
- net /RTS: track 0.00 -> 44.5 mm, vias 0 -> 2
- net /IO0: track 0.00 -> 42.3 mm
- net Net-(D2-A): track 0.00 -> 37.1 mm, vias 0 -> 2
- net /supply/TXD: track 0.00 -> 34.7 mm, vias 0 -> 3
- net Net-(U1-IO12): track 0.00 -> 28.3 mm, vias 0 -> 2
- net Net-(P1-D-): track 0.00 -> 26.5 mm, vias 0 -> 2
- net Net-(J1-Pin_1): track 0.00 -> 21.3 mm, vias 0 -> 1
- net Net-(Q1-B): track 0.00 -> 21.3 mm, vias 0 -> 2
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
Commit message: init
Parts:
- moved L1 32.6 mm to (143.0, 93.0), turned to 90 degrees
- moved C3 24.2 mm to (143.0, 86.5), turned to 90 degrees
- moved R6 23.9 mm to (143.5, 75.5)
- moved R9 22.9 mm to (130.5, 86.5), turned to 90 degrees
- moved C2 22.5 mm to (139.0, 86.5), turned to 90 degrees
- moved R1 21.9 mm to (146.5, 70.0)
- moved D2 20.1 mm to (122.3, 80.5)
- moved R4 18.1 mm to (139.5, 75.5)
- moved C6 17.9 mm to (136.5, 81.5), turned to 0 degrees
- moved R2 17.7 mm to (142.0, 64.5), turned to -90 degrees
- moved C7 17.7 mm to (151.0, 71.5)
- moved Q2 17.0 mm to (138.4, 70.6), turned to 90 degrees
- moved Q1 16.8 mm to (146.5, 64.5)
- moved R3 15.2 mm to (126.0, 75.5)
- moved C1 14.5 mm to (130.0, 75.5), turned to -90 degrees
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Routing:
- net Net-(U4-VBUS): track 70.8 -> 16.8 mm, vias 3 -> 2
- net Net-(U1-LNA_IN): track 15.7 -> 57.6 mm
- net Net-(C2-Pad1): track 48.0 -> 9.85 mm, vias 4 -> 0
- net +3.3V: track 181.8 -> 146.6 mm, vias 6 -> 10
- net Net-(Q2-B): track 45.3 -> 10.5 mm, vias 2 -> 0
- net /supply/RXD: track 17.3 -> 50.4 mm, vias 2 -> 0
- net /CTS: track 15.5 -> 40.6 mm
- net /supply/DTR: track 13.1 -> 37.9 mm, vias 0 -> 2
- net +5V: track 61.4 -> 47.0 mm, vias 4 -> 2
- net Net-(U4-D+): track 7.98 -> 20.2 mm, vias 0 -> 2
- net Net-(U4-~{SUSPEND}): track 8.57 -> 19.4 mm, vias 0 -> 2
- net Net-(P1-D+): track 21.1 -> 30.8 mm
- net Net-(J1-Pin_5): track 16.5 -> 6.98 mm, vias 0 -> 1
- net /IO0: track 42.3 -> 33.3 mm, vias 0 -> 2
- net Net-(U1-IO12): track 28.3 -> 19.4 mm
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- added copper zone on F.Cu, net GND
Other:
- board size 37 x 40 mm -> 38 x 40 mm
