File: kicad/esp32-clock.kicad_pcb (KiCad board)
At the start: 2 copper layers, 38 x 40 mm, 36 parts, among them J1 Conn_01x07_Socket, P1 USB_C_Plug_USB2.0, Q1 BCW66G, Q2 BCW66G, SW1 RESET, SW2 BOOT, U1 ESP32-PICO-V3, U2 USBLC6-2P6, U3 AMS1117-3.3, U4 CP2102N-Axx-xQFN28

Commit message: init
Parts:
- added C10: 100nF, Capacitor_SMD:C_1206_3216Metric, F.Cu at (137.2, 67.3)
- added C8: 100pF, Capacitor_SMD:C_1206_3216Metric, F.Cu at (125.7, 61.0)
- added C9: 10µF, Capacitor_SMD:C_1206_3216Metric, F.Cu at (125.7, 86.4)
- added D4: red, Diode_SMD:D_0603_1608Metric, F.Cu at (154.5, 77.5)
- added D5: red, Diode_SMD:D_0603_1608Metric, F.Cu at (133.3, 82.5)
- added J2: Conn_01x02_Socket, Connector_JST:JST_XH_B2B-XH-A_1x02_P2.50mm_Vertical, F.Cu at (150.5, 66.0)
- added R13: 2K, Resistor_SMD:R_1206_3216Metric, F.Cu at (135.9, 87.6)
- added R14: 1K, Resistor_SMD:R_1206_3216Metric, F.Cu at (142.2, 67.3)
- added R15: 100, Resistor_SMD:R_1206_3216Metric, F.Cu at (132.1, 68.6)
- added U5: U8205A, Package_TO_SOT_SMD:SOT-23-6, F.Cu at (137.2, 63.5)
- added U6: DW01A, Package_TO_SOT_SMD:SOT-23-6, F.Cu at (132.1, 63.5)
- added U7: AMS1117-3.3, Package_TO_SOT_SMD:SOT-223-3_TabPin2, F.Cu at (123.2, 78.7)
- added U8: Switch, PCM_yvolodym:Switch, F.Cu at (148.9, 72.4)
- C6: value 100nF -> 10µF
- D1, D3: value LED -> green
- D2: value LED -> blue
- R10: value 2K -> 1K
- R11: value 2 K -> 1K
- R12: value 10 K -> 2K
- R4: value 1K -> 10K
- R5: value 10K -> 1K
- R8: value 47 K -> 470
- R9: value 100 K -> 470
- U2: value USBLC6-2P6 -> CH340C; footprint Package_TO_SOT_SMD:SOT-23-6 -> Package_SO:SOIC-16_3.9x9.9mm_P1.27mm
- U3: value AMS1117-3.3 -> TP4056-42-ESOP8; footprint Package_TO_SOT_SMD:SOT-223-3_TabPin2 -> Package_SO:SOIC-8-1EP_3.9x4.9mm_P1.27mm_EP2.41x3.3mm_ThermalVias
- U4: value CP2102N-Axx-xQFN28 -> USBLC6-2P6; footprint Package_DFN_QFN:QFN-28-1EP_5x5mm_P0.5mm_EP3.35x3.35mm -> Package_TO_SOT_SMD:SOT-23-6
- moved C5 37.2 mm to (148.6, 59.7), turned to 90 degrees
- moved SW1 34.2 mm to (129.5, 91.4)
- moved R2 33.5 mm to (132.1, 96.5), turned to 0 degrees
- moved L1 31.3 mm to (119.4, 72.4), turned to -90 degrees
- moved H1 30.7 mm to (121.9, 58.4)
- moved R5 30.1 mm to (143.5, 96.5), turned to 0 degrees
- moved H2 30.0 mm to (152.4, 58.4)
- moved D2 29.7 mm to (147.3, 96.5), turned to -90 degrees
- moved Q1 29.3 mm to (138.4, 92.7)
- moved C1 29.0 mm to (152.4, 94.0), turned to 0 degrees
- moved U4 29.0 mm to (142.2, 63.5), turned to 90 degrees
- moved R1 25.6 mm to (134.6, 92.7), turned to -90 degrees
- moved C7 25.4 mm to (129.5, 85.1), turned to -90 degrees
- moved D1 24.8 mm to (147.3, 94.0), turned to 0 degrees
- moved R7 24.6 mm to (141.0, 88.9), turned to 0 degrees
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Connections:
- net Net-(U4-D+) renamed /Supply_2/D-
- C7 pad 1: +3.3V -> +5V
- D3 pad 1: GND -> Net-(D3-K)
- D3 pad 2: Net-(D3-A) -> +5V
- Q2 pad 3: /supply/DTR -> /DTR
- R10 pad 1: +5V -> Net-(U3-~{STDBY})
- R10 pad 2: Net-(D3-A) -> Net-(D3-K)
- R11 pad 1: +3.3V -> Net-(U3-~{CHRG})
- R11 pad 2: Net-(U4-~{RST}) -> Net-(D4-K)
- R12 pad 1: Net-(U4-~{SUSPEND}) -> GND
- R12 pad 2: GND -> Net-(U3-PROG)
- R3 pad 1: /supply/TXD -> /RXD0
- R4 pad 1: /supply/RXD -> +3.3V
- R4 pad 2: Net-(D2-A) -> /IO0
- R5 pad 1: +3.3V -> /TXD0
- R5 pad 2: /IO0 -> Net-(D2-A)
- R6 pad 1: /supply/DTR -> /DTR
- R8 pad 1: +5V -> Net-(U2-TXD)
- R8 pad 2: Net-(U4-VBUS) -> /RXD0
- R9 pad 1: Net-(U4-VBUS) -> Net-(U2-RXD)
- R9 pad 2: GND -> /TXD0
- U1 pad 32: unconnected-(U1-SD0-Pad32) -> Net-(J1-Pin_5)
- U1 pad 33: unconnected-(U1-SD1-Pad33) -> Net-(J1-Pin_4)
- U1 pad 35: Net-(J1-Pin_5) -> unconnected-(U1-NC-Pad35)
- U1 pad 36: Net-(J1-Pin_4) -> unconnected-(U1-NC-Pad36)
- U1 pad 40: /supply/TXD -> /RXD0
- U1 pad 41: /supply/RXD -> /TXD0
- U2 pad 1: Net-(P1-D+) -> GND
- U2 pad 2: GND -> Net-(U2-TXD)
- U2 pad 3: Net-(P1-D-) -> Net-(U2-RXD)
- U2 pad 4: Net-(U4-D-) -> +3.3V
- U2 pad 5: +5V -> /Supply_2/D+
- U3 pad 2: +3.3V -> Net-(U3-PROG)
- U3 pad 3: +5V -> GND
- U4 pad 1: unconnected-(U4-~{DCD}-Pad1) -> Net-(P1-D+)
- U4 pad 2: unconnected-(U4-~{RI}/CLK-Pad2) -> GND
- U4 pad 3: GND -> Net-(P1-D-)
- U4 pad 5: Net-(U4-D-) -> +5V
- U4 pad 6: +3.3V -> /Supply_2/D+
Routing:
- net GND: track 197.7 -> 0.00 mm, vias 4 -> 0
- net +3.3V: track 146.6 -> 0.00 mm, vias 10 -> 0
- net Net-(U1-LNA_IN): track 57.6 -> 0.00 mm, vias 2 -> 0
- net /supply/RXD: track 50.4 -> 0.00 mm
- net /RTS: track 47.3 -> 0.00 mm, vias 3 -> 0
- net +5V: track 47.0 -> 0.00 mm, vias 2 -> 0
- net /EN: track 46.3 -> 0.00 mm, vias 2 -> 0
- net /CTS: track 40.6 -> 0.00 mm, vias 2 -> 0
- net /supply/TXD: track 39.7 -> 0.00 mm, vias 5 -> 0
- net /supply/DTR: track 37.9 -> 0.00 mm, vias 2 -> 0
- net Net-(D2-A): track 33.9 -> 0.00 mm, vias 2 -> 0
- net /IO0: track 33.3 -> 0.00 mm, vias 2 -> 0
- net Net-(P1-D+): track 30.8 -> 0.00 mm, vias 2 -> 0
- net Net-(J1-Pin_1): track 27.9 -> 0.00 mm, vias 1 -> 0
- net Net-(P1-D-): track 24.4 -> 0.00 mm, vias 2 -> 0
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- removed copper zone on F.Cu, net GND
Other:
- board size 38 x 40 mm -> 38 x 43 mm

Commit message: init
Parts:
- added J3: GND, TestPoint:TestPoint_THTPad_2.5x2.5mm_Drill1.2mm, F.Cu at (154.0, 63.9)
- J2: value Conn_01x02_Socket -> +3.3; footprint Connector_JST:JST_XH_B2B-XH-A_1x02_P2.50mm_Vertical -> TestPoint:TestPoint_THTPad_2.5x2.5mm_Drill1.2mm
- moved J2 2.92 mm to (147.6, 66.5)
- moved D4 0.70 mm to (154.0, 77.9)
- moved Q2 0.53 mm to (143.8, 93.2)
- moved U7 0.53 mm to (123.5, 79.2)
- moved C7 0.53 mm to (129.8, 85.5)
- moved D1 0.53 mm to (147.6, 94.4)
- moved D2 0.53 mm to (147.6, 97.0)
- moved J1 0.53 mm to (129.8, 58.9)
- moved R10 0.53 mm to (147.6, 77.9)
- moved R13 0.53 mm to (136.2, 88.1)
- moved R5 0.53 mm to (143.8, 97.0)
- moved R6 0.53 mm to (136.2, 81.7)
- moved SW1 0.53 mm to (129.8, 91.9)
- moved U2 0.53 mm to (140.0, 74.1)
- moved C2 0.53 mm to (126.0, 93.2)
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Connections:
- U8 pad 2: Net-(J2-Pin_2) -> Net-(J3-Pin_1)
