File: kicad/esp32-clock.kicad_sch (KiCad schematic)
At the start: 0 parts

Commit message: init
Parts:
- added C3, C6: 0.1µF, Capacitor_SMD:C_0201_0603Metric, symbol Device:C
- added R6: 10k, Resistor_SMD:R_0201_0603Metric, symbol Device:R
- added SW1: RESET, Button_Switch_SMD:SW_SPST_CK_KMS2xxGP, symbol Switch:CK_KMS2xxG
- added SW2: BOOT, Button_Switch_SMD:SW_SPST_CK_KMS2xxGP, symbol Switch:CK_KMS2xxG
- added U3: ESP-12E, RF_Module:ESP-12E, symbol RF_Module:ESP-12E
Connections:
- new net: C6.1, SW2.1, U3.18 (GPIO0)
- new net: C3.1, R6.2, SW1.2, U3.3 (EN)
- new net +3.3V: R6.1, U3.8 (VCC)
- new net GND: C3.2, C6.2, SW1.1, SW1.SH (B), SW2.SH (B), U3.15 (GND)

Commit message: init
Other:
- sheet supply ports: added USB_D_N; removed none
Changed lines of the file:
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@@
+			)
+		)
+		(pin "USB_D_N" input
+			(at 191.77 41.91 180)
+			(effects
+				(font
+					(size 1.27 1.27)
+				)
+				(justify left)
 			)
 		)

Commit message: init
Connections:
- net supply/RXD: now reaches U3.21 (GPIO3/RXD)
- net supply/TXD: now reaches U3.22 (GPIO1/TXD)
Other:
- sheet supply ports: added RTS, RXD, TXD; removed USB_D_N
Changed lines of the file:
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@@
+	(wire
+		(pts
+			(xy 104.14 75.565) (xy 118.11 75.565)
+		)
+		(stroke
+			(width 0)
+			(type default)
+		)
+	)
+	(wire
+		(pts
+			(xy 104.14 70.485) (xy 114.935 70.485)
+		)
+		(stroke
+			(width 0)
+			(type default)
+		)
+	)
 	(wire
 		(pts
@@
 	(wire
 		(pts
+			(xy 114.935 45.72) (xy 191.77 45.72)
+		)
+		(stroke
+			(width 0)
+			(type default)
+		)
+	)
+	(wire
+		(pts
 			(xy 54.61 73.025) (xy 54.61 74.295)
 		)
@@
 	(wire
 		(pts
+			(xy 118.11 51.435) (xy 191.77 51.435)
+		)
+		(stroke
+			(width 0)
+			(type default)
+		)
+	)
+	(wire
+		(pts
 			(xy 121.285 67.945) (xy 121.285 74.93)
 		)
@@
 	(wire
 		(pts
+			(xy 114.935 70.485) (xy 114.935 45.72)
+		)
+		(stroke
+			(width 0)
+			(type default)
+		)
+	)
+	(wire
+		(pts
 			(xy 121.285 67.945) (xy 128.905 67.945)
 		)
@@
 		(pts
 			(xy 33.655 84.455) (xy 41.91 84.455)
+		)
+		(stroke
+			(width 0)
+			(type default)
+		)
+	)
+	(wire
+		(pts
+			(xy 118.11 75.565) (xy 118.11 51.435)
 		)
 		(stroke
@@
 			)
 		)
-		(pin "USB_D_N" input
-			(at 191.77 41.91 180)
-			(effects
-				(font
+		(pin "RTS" input
+			(at 191.77 40.64 180)
+			(effects
+				(font
+					(size 1.27 1.27)
+				)
+				(justify left)
+			)
+		)
+		(pin "TXD" input
+			(at 191.77 45.72 180)
+			(effects
+				(font
+					(size 1.27 1.27)
+				)
+				(justify left)
+			)
+		)
+		(pin "RXD" input
+			(at 191.77 51.435 180)
+			(effects
+				(font

Commit message: init
Parts:
- C1: renamed from C3; footprint Capacitor_SMD:C_0201_0603Metric -> Capacitor_SMD:C_1206_3216Metric
- C2: renamed from C6; footprint Capacitor_SMD:C_0201_0603Metric -> Capacitor_SMD:C_1206_3216Metric
- R1: renamed from R6; footprint Resistor_SMD:R_0201_0603Metric -> Resistor_SMD:R_2816_7142Metric
- renumbered U3 to U1
Changed lines of the file:
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@@
 		(dnp no)
 		(fields_autoplaced yes)
-		(property "Reference" "U3"
+		(property "Reference" "U1"
 			(at 91.0941 60.96 0)
 			(effects
@@
 			(project ""
 				(path "/705cc6fa-d5d2-496f-be92-82c69a6f5679"
-					(reference "U3")
+					(reference "U1")
 					(unit 1)
 				)
@@
 		(on_board yes)
 		(dnp no)
-		(property "Reference" "C6"
+		(property "Reference" "C2"
 			(at 125.095 77.4699 0)
 			(effects
@@
 			)
 		)
-		(property "Footprint" "Capacitor_SMD:C_0201_0603Metric"
+		(property "Footprint" "Capacitor_SMD:C_1206_3216Metric"
 			(at 122.2502 82.55 0)
 			(effects
@@
 			(project "esp32-clock"
 				(path "/705cc6fa-d5d2-496f-be92-82c69a6f5679"
-					(reference "C6")
+					(reference "C2")
 					(unit 1)
 				)
@@
 		(dnp no)
 		(fields_autoplaced yes)
-		(property "Reference" "#PWR09"
+		(property "Reference" "#PWR03"
 			(at 88.9 66.675 0)
 			(effects
@@
 			(project ""
 				(path "/705cc6fa-d5d2-496f-be92-82c69a6f5679"
-					(reference "#PWR09")
+					(reference "#PWR03")
 					(unit 1)
 				)
@@
 		(dnp no)
 		(fields_autoplaced yes)
-		(property "Reference" "#PWR012"
+		(property "Reference" "#PWR01"
 			(at 41.91 93.345 0)
 			(effects
@@
 			(project ""
 				(path "/705cc6fa-d5d2-496f-be92-82c69a6f5679"
-					(reference "#PWR012")
+					(reference "#PWR01")
 					(unit 1)
 				)
@@
 		(dnp no)
 		(fields_autoplaced yes)
-		(property "Reference" "#PWR010"
+		(property "Reference" "#PWR04"
 			(at 88.9 107.315 0)
 			(effects
@@
 			(project ""
 				(path "/705cc6fa-d5d2-496f-be92-82c69a6f5679"
-					(reference "#PWR010")
+					(reference "#PWR04")
 					(unit 1)
 				)
@@
 		(dnp no)
 		(fields_autoplaced yes)
-		(property "Reference" "#PWR011"
+		(property "Reference" "#PWR05"
 			(at 133.985 90.805 0)
 			(effects
@@
 			(project ""
 				(path "/705cc6fa-d5d2-496f-be92-82c69a6f5679"
-					(reference "#PWR011")
+					(reference "#PWR05")
 					(unit 1)
 				)
@@
 		(dnp no)
 		(fields_autoplaced yes)
-		(property "Reference" "#PWR013"
+		(property "Reference" "#PWR02"
 			(at 54.61 64.135 0)
 			(effects
@@
 			(project ""
 				(path "/705cc6fa-d5d2-496f-be92-82c69a6f5679"
-					(reference "#PWR013")
+					(reference "#PWR02")
 					(unit 1)
 				)
@@
 		(dnp no)
 		(fields_autoplaced yes)
-		(property "Reference" "C3"
+		(property "Reference" "C1"
 			(at 58.42 76.8349 0)
 			(effects
@@
 			)
 		)
-		(property "Footprint" "Capacitor_SMD:C_0201_0603Metric"
+		(property "Footprint" "Capacitor_SMD:C_1206_3216Metric"
 			(at 55.5752 81.915 0)
 			(effects
@@
 			(project ""
 				(path "/705cc6fa-d5d2-496f-be92-82c69a6f5679"
-					(reference "C3")
+					(reference "C1")
 					(unit 1)
 				)
@@
 		(dnp no)
 		(fields_autoplaced yes)
-		(property "Reference" "R6"
+		(property "Reference" "R1"
 			(at 57.15 62.8649 0)
 			(effects
@@
 			)
 		)
-		(property "Footprint" "Resistor_SMD:R_0201_0603Metric"
+		(property "Footprint" "Resistor_SMD:R_2816_7142Metric"
 			(at 52.832 64.135 90)
 			(effects
@@
 			(project ""
 				(path "/705cc6fa-d5d2-496f-be92-82c69a6f5679"
-					(reference "R6")
-					(unit 1)
-				)
+					(reference "R1")
+					(unit 1)
+				)

Commit message: init
Connections:
- no-connect marks 0 -> 1
Changed lines of the file:
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@@
 		(color 0 0 0 0)
+	)
+	(no_connect
+		(at 139.065 67.945)
 	)
 	(wire

Commit message: init
Parts:
- R1: footprint Resistor_SMD:R_2816_7142Metric -> Resistor_SMD:R_1206_3216Metric; LCSC (none) -> C1489
Connections:
- no-connect marks 1 -> 17
Other:
- sheet supply ports: added none; removed RTS
- moved on the sheet: C1, C2, R1, SW1, SW2, U1

Commit message: init
Changed lines of the file:
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@@
+	)
+	(junction
+		(at 121.92 82.55)
+		(diameter 0)
+		(color 0 0 0 0)
 	)
 	(junction
@@
 	)
 	(junction
+		(at 64.77 73.66)
+		(diameter 0)
+		(color 0 0 0 0)
+	)
+	(junction
 		(at 134.62 82.55)
 		(diameter 0)
@@
 	(wire
 		(pts
+			(xy 121.92 82.55) (xy 121.92 85.09)
+		)
+		(stroke
+			(width 0)
+			(type default)
+		)
+	)
+	(wire
+		(pts
 			(xy 54.61 82.55) (xy 54.61 85.09)
 		)
@@
 	(wire
 		(pts
+			(xy 64.77 67.31) (xy 64.77 73.66)
+		)
+		(stroke
+			(width 0)
+			(type default)
+		)
+	)
+	(wire
+		(pts
 			(xy 104.14 76.2) (xy 118.11 76.2)
 		)
@@
 	(wire
 		(pts
-			(xy 73.66 73.66) (xy 54.61 73.66)
+			(xy 73.66 73.66) (xy 64.77 73.66)
 		)
 		(stroke
@@
 	(wire
 		(pts
+			(xy 64.77 73.66) (xy 54.61 73.66)
+		)
+		(stroke
+			(width 0)
+			(type default)
+		)
+	)
+	(wire
+		(pts
 			(xy 36.83 73.66) (xy 34.29 73.66)
 		)
@@
 			(width 0)
 			(type default)
+		)
+	)
+	(symbol
+		(lib_id "power:PWR_FLAG")
+		(at 64.77 67.31 0)
+		(unit 1)
+		(exclude_from_sim no)
+		(in_bom yes)
+		(on_board yes)
+		(dnp no)
+		(fields_autoplaced yes)
+		(property "Reference" "#FLG03"
+			(at 64.77 65.405 0)
+			(effects
+				(font
+					(size 1.27 1.27)
+				)
+				(hide yes)
+			)
+		)
+		(property "Value" "PWR_FLAG"
+			(at 64.77 62.23 0)
+			(effects
+				(font
+					(size 1.27 1.27)
+				)
+			)
+		)
+		(property "Footprint" ""
+			(at 64.77 67.31 0)
+			(effects
+				(font
+					(size 1.27 1.27)
+				)
+				(hide yes)
+			)
+		)
+		(property "Datasheet" "~"
+			(at 64.77 67.31 0)
+			(effects
+				(font
+					(size 1.27 1.27)
+				)
+				(hide yes)
+			)
+		)
+		(property "Description" "Special symbol for telling ERC where power comes from"
+			(at 64.77 67.31 0)
+			(effects
+				(font
+					(size 1.27 1.27)
+				)
+				(hide yes)
+			)
+		)
+		(pin "1"
+		)
+		(instances
+			(project ""
+				(path "/705cc6fa-d5d2-496f-be92-82c69a6f5679"
+					(reference "#FLG03")
+					(unit 1)
+				)
+			)
 		)
 	)
@@
 					(unit 1)
 				)
+			)
+		)
+	)
+	(symbol
+		(lib_id "power:PWR_FLAG")
+		(at 121.92 85.09 180)
+		(unit 1)
+		(exclude_from_sim no)
+		(in_bom yes)
+		(on_board yes)
+		(dnp no)
+		(fields_autoplaced yes)
+		(property "Reference" "#FLG04"
+			(at 121.92 86.995 0)
+			(effects
+				(font
+					(size 1.27 1.27)
+				)
+				(hide yes)
+			)
+		)
+		(property "Value" "PWR_FLAG"
+			(at 121.92 90.17 0)
+			(effects
+				(font
+					(size 1.27 1.27)
+				)
+			)
+		)
+		(property "Footprint" ""
+			(at 121.92 85.09 0)
+			(effects
+				(font
+					(size 1.27 1.27)
+				)
+				(hide yes)
+			)
+		)
+		(property "Datasheet" "~"
+			(at 121.92 85.09 0)
+			(effects
+				(font
+					(size 1.27 1.27)
+				)
+				(hide yes)
+			)
+		)
+		(property "Description" "Special symbol for telling ERC where power comes from"
+			(at 121.92 85.09 0)
+			(effects
+				(font
+					(size 1.27 1.27)
+				)
+				(hide yes)
+			)
+		)
+		(pin "1"
+		)
+		(instances
+			(project "esp32-clock"
+				(path "/705cc6fa-d5d2-496f-be92-82c69a6f5679"
+					(reference "#FLG04")
+					(unit 1)
+				)

Commit message: init
Connections:
- net GND: now also SW2.2
- no-connect marks 17 -> 16
Changed lines of the file:
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@@
-	)
-	(no_connect
-		(at 139.7 68.58)
 	)
 	(no_connect
@@
 	(wire
 		(pts
+			(xy 139.7 82.55) (xy 134.62 82.55)
+		)
+		(stroke
+			(width 0)
+			(type default)
+		)
+	)
+	(wire
+		(pts
 			(xy 64.77 67.31) (xy 64.77 73.66)
 		)
@@
 		)
 		(stroke
+			(width 0)
+			(type default)
+		)
+	)
+	(wire
+		(pts
+			(xy 139.7 68.58) (xy 139.7 82.55)
+		)
+		(stroke
