File: kicad/esp32-clock.kicad_sch (KiCad schematic)
At the start: 7 parts, among them J3 Conn_01x06_Pin, SW1 RESET, SW2 BOOT, U1 ESP-12E

Commit message: init
Parts:
- removed J3: Conn_01x06_Pin, Connector_PinHeader_2.54mm:PinHeader_1x06_P2.54mm_Vertical, symbol Connector:Conn_01x06_Pin
- added H1, H2, H3, H4: MountingHole, MountingHole:MountingHole_2.2mm_M2_DIN965_Pad, symbol Mechanical:MountingHole
- added U?: ESP32-PICO-V3, Package_DFN_QFN:QFN-48-1EP_7x7mm_P0.5mm_EP5.15x5.15mm, symbol PCM_Espressif:ESP32-PICO-V3
Connections:
- new net: U?.1 (VDDA), U?.43 (VDDA), U?.46 (VDDA)
- new net: U?.3 (VDD3P3), U?.4 (VDD3P3)

Commit message: init
Parts:
- removed U1: ESP-12E, RF_Module:ESP-12E, symbol RF_Module:ESP-12E
- added J1: Conn_01x07_Socket, Connector_PinSocket_2.54mm:PinSocket_1x07_P2.54mm_Vertical, symbol Connector:Conn_01x07_Socket
- C1, C2: value 0.1µF -> 0,1µF
- R1: value 10k -> 10K; LCSC C1489 -> (none)
- gave numbers to parts that had none: 1
Connections:
- net +3.3V: now also U1.1 (VDDA), U1.3 (VDD3P3), U1.4 (VDD3P3), U1.43 (VDDA), U1.46 (VDDA), J1.7 (Pin_7)
- net GND: now also U1.49 (GND), J1.6 (Pin_6)
- net supply/RXD: now also U1.40 (U0RXD/GPIO3)
- net supply/TXD: now also U1.41 (U0TXD/GPIO1)
- net at C2.1, SW2.1: now also U1.23 (GPIO0/BOOT/ADC2_CH1)
- net EN: now reaches C1.1, R1.2, SW1.2
- net EN: now also U1.9 (CHIP_PU)
- net RTS: now reaches U1.20 (MTCK/GPIO13/ADC2_CH4)
- net CTS: now reaches U1.21 (MTDO/GPIO15/ADC2_CH3)
- net at U1.27 (GPIO20): now also J1.2 (Pin_2)
- net at U1.29 (SD_DATA_3/GPIO10): now also J1.5 (Pin_5)
- net at U1.38 (GPIO19): now also J1.1 (Pin_1)
- net at U1.39 (GPIO22): now also J1.4 (Pin_4)
- net at U1.42 (GPIO21): now also J1.3 (Pin_3)
- no-connect marks 12 -> 25
Other:
- note added: "CS"
- note added: "DC"
- note added: "GND"
- note added: "RST"
- note added: "SCL"
- note added: "SOA [MOSI]"
- note added: "VCC"
- moved on the sheet: SW1, SW2, U1

Commit message: init
Parts:
- removed H4: MountingHole, MountingHole:MountingHole_2.2mm_M2_DIN965_Pad, symbol Mechanical:MountingHole
- added C8: 2,7pF, Capacitor_SMD:C_1206_3216Metric, symbol Device:C
- added C9: 4,7pF, Capacitor_SMD:C_1206_3216Metric, symbol Device:C
- added L1: 1,6nH, symbol Device:L
- added TP1: TestPoint_2Pole, symbol Connector:TestPoint_2Pole
Connections:
- net GND: now also C8.2, L1.2, TP1.1
- net at U1.2 (LNA_IN): now also C9.2, L1.1
- new net: C8.1, C9.1, TP1.2
- no-connect marks 25 -> 24

Commit message: init
Parts:
- removed H1: MountingHole, MountingHole:MountingHole_2.2mm_M2_DIN965_Pad, symbol Mechanical:MountingHole
- removed TP1: TestPoint_2Pole, symbol Connector:TestPoint_2Pole
- added TP1, TP2: TestPoint, TestPoint:TestPoint_Pad_3.0x3.0mm, symbol Connector:TestPoint
- renumbered C8 to C2, C9 to C3, C2 to C4
Connections:
- net GND: now also TP1.1
- net at C2.1, C3.1: now also TP2.1

Commit message: init
Parts:
- L1: footprint (none) -> Inductor_SMD:L_1206_3216Metric_Pad1.42x1.75mm_HandSolder
- SW1, SW2: footprint Button_Switch_SMD:SW_SPST_CK_KMS2xxGP -> Button_Switch_SMD:SW_Push_1P1T_NO_CK_KMR2
- renumbered H2 to H1, H3 to H2
Changed lines of the file:
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@@
 		(on_board yes)
 		(dnp no)
-		(property "Reference" "H3"
+		(property "Reference" "H2"
 			(at 55.88 163.8299 0)
 			(effects
@@
 			(project "esp32-clock"
 				(path "/705cc6fa-d5d2-496f-be92-82c69a6f5679"
-					(reference "H3")
+					(reference "H2")
 					(unit 1)
 				)
@@
 			)
 		)
-		(property "Footprint" ""
+		(property "Footprint" "Inductor_SMD:L_1206_3216Metric_Pad1.42x1.75mm_HandSolder"
 			(at 64.77 44.45 0)
 			(effects
@@
 			)
 		)
-		(property "Footprint" "Button_Switch_SMD:SW_SPST_CK_KMS2xxGP"
+		(property "Footprint" "Button_Switch_SMD:SW_Push_1P1T_NO_CK_KMR2"
 			(at 233.68 76.2 0)
 			(effects
@@
 		(on_board yes)
 		(dnp no)
-		(property "Reference" "H2"
+		(property "Reference" "H1"
 			(at 45.72 163.8299 0)
 			(effects
@@
 			(project "esp32-clock"
 				(path "/705cc6fa-d5d2-496f-be92-82c69a6f5679"
-					(reference "H2")
+					(reference "H1")
 					(unit 1)
 				)
@@
 			)
 		)
-		(property "Footprint" "Button_Switch_SMD:SW_SPST_CK_KMS2xxGP"
+		(property "Footprint" "Button_Switch_SMD:SW_Push_1P1T_NO_CK_KMR2"
 			(at 25.4 73.66 0)
 			(effects

Commit message: init
Parts:
- C1, C4: value 0,1µF -> 100nF
Changed lines of the file:
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@@
 			)
 		)
-		(property "Value" "0,1µF"
+		(property "Value" "100nF"
 			(at 41.91 87.6299 0)
 			(effects
@@
 			)
 		)
-		(property "Value" "0,1µF"
+		(property "Value" "100nF"
 			(at 227.33 88.8999 0)
 			(effects

Commit message: init
Other:
- moved on the sheet: C1
Changed lines of the file:
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@@
+	(wire
+		(pts
+			(xy 38.1 87.63) (xy 38.1 90.17)
+		)
+		(stroke
+			(width 0)
+			(type default)
+		)
+	)
 	(wire
 		(pts
@@
 	(wire
 		(pts
-			(xy 38.1 78.74) (xy 38.1 82.55)
+			(xy 38.1 78.74) (xy 38.1 80.01)
 		)
 		(stroke
@@
 	(symbol
 		(lib_id "Device:C")
-		(at 38.1 86.36 0)
+		(at 38.1 83.82 0)
 		(unit 1)
 		(exclude_from_sim no)
@@
 		(fields_autoplaced yes)
 		(property "Reference" "C1"
+			(at 41.91 82.5499 0)
+			(effects
+				(font
+					(size 1.27 1.27)
+				)
+				(justify left)
+			)
+		)
+		(property "Value" "100nF"
 			(at 41.91 85.0899 0)
 			(effects
@@
 			)
 		)
-		(property "Value" "100nF"
-			(at 41.91 87.6299 0)
-			(effects
-				(font
-					(size 1.27 1.27)
-				)
-				(justify left)
-			)
-		)
 		(property "Footprint" "Capacitor_SMD:C_1206_3216Metric"
-			(at 39.0652 90.17 0)
+			(at 39.0652 87.63 0)
 			(effects
 				(font
@@
 		)
 		(property "Datasheet" "~"
-			(at 38.1 86.36 0)
+			(at 38.1 83.82 0)
 			(effects
 				(font
@@
 		)
 		(property "Description" "Unpolarized capacitor"
-			(at 38.1 86.36 0)
-			(effects
-				(font
+			(at 38.1 83.82 0)
+			(effects
+				(font

Commit message: init
Parts:
- added D1, D2: LED, Diode_SMD:D_0603_1608Metric, symbol Device:LED
- added R2, R3: 1K, Resistor_SMD:R_1206_3216Metric, symbol Device:R
Connections:
- net GND: now also D1.1 (K), D2.1 (K)
- net supply/RXD: now also R3.1
- net supply/TXD: now also R2.1
- new net: D2.2 (A), R3.2
- new net: D1.2 (A), R2.2
