File: kicad/esp32-clock.kicad_sch (KiCad schematic)
At the start: 18 parts, among them J1 Conn_01x07_Socket, SW1 RESET, SW2 BOOT, U1 ESP32-PICO-V3

Commit message: init
Parts:
- added R4: 10K, Resistor_SMD:R_1206_3216Metric, symbol Device:R
Connections:
- net +3.3V: now also R4.1
- net IO0: now reaches C4.1, SW2.1, U1.23 (GPIO0/BOOT/ADC2_CH1)
- net IO0: now also R4.2
Other:
- sheet supply ports: added CTS, EN, IO0, RTS; removed none

Commit message: init
Parts:
- removed TP1: TestPoint, TestPoint:TestPoint_Pad_3.0x3.0mm, symbol Connector:TestPoint
- added R2: 10K, Resistor_SMD:R_1206_3216Metric, symbol Device:R
- renumbered R2 to R3, R3 to R4, R4 to R5, TP2 to TP1
Connections:
- net +3.3V: now also U1.19 (VDD3P3_RTC), U1.37 (VDD3P3_CPU), R2.2
- net at U1.18 (MTDI/GPIO12/ADC2_CH5): now also R2.1
- no-connect marks 24 -> 21

Commit message: init
Parts:
- removed U1: ESP32-PICO-V3, Package_DFN_QFN:QFN-48-1EP_7x7mm_P0.5mm_EP5.15x5.15mm, symbol PCM_Espressif:ESP32-PICO-V3
- added U1: ESP32-PICO-V3, Package_DFN_QFN:QFN-48-1EP_7x7mm_P0.5mm_EP5.3x5.3mm, symbol MCU_Espressif:ESP32-PICO-V3
Connections:
- net +3.3V: now also U1.1 (VDDA), U1.19 (VDD3P3_RTC), U1.3 (VDDA3P3), U1.37 (VDD3P3_CPU), U1.4 (VDDA3P3), U1.43 (VDDA), U1.46 (VDDA)
- net CTS: now also U1.21 (IO15)
- net EN: now also U1.9 (EN)
- net GND: now also U1.49 (GND)
- net IO0: now also U1.23 (IO0)
- net RTS: now also U1.20 (IO13)
- net supply/RXD: now also U1.40 (U0RXD/IO3)
- net supply/TXD: now also U1.41 (U0TXD/IO1)
- net at C3.2, L1.1: now also U1.2 (LNA_IN)
- net at R2.1: now also U1.18 (IO12)
- net at J1.2 (Pin_2): now also U1.34 (IO5)
- net at J1.5 (Pin_5): now also U1.35 (IO18)
- net at J1.1 (Pin_1): now also U1.39 (IO22)
- net at J1.4 (Pin_4): now also U1.36 (IO23)
- net at J1.3 (Pin_3): now also U1.42 (IO21)
- no-connect marks 21 -> 24
Other:
- moved on the sheet: C1, C2, C3, C4, J1, L1, R1, R2, R5, SW1, SW2, TP1

Commit message: init
Connections:
- net supply/RXD: now also U1.41 (U0TXD/IO1); no longer U1.40 (U0RXD/IO3)
- net supply/TXD: now also U1.40 (U0RXD/IO3); no longer U1.41 (U0TXD/IO1)
Changed lines of the file:
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@@
 	(text "RST"
 		(exclude_from_sim no)
-		(at 179.07 114.3 0)
+		(at 179.578 114.3 0)
 		(effects
 			(font
@@
 	(text "DC"
 		(exclude_from_sim no)
-		(at 179.07 119.38 0)
+		(at 179.324 119.38 0)
 		(effects
 			(font
@@
 	(text "SCL"
 		(exclude_from_sim no)
-		(at 180.34 124.46 0)
+		(at 179.832 124.46 0)
 		(effects
 			(font
@@
 	(text "VCC"
 		(exclude_from_sim no)
-		(at 180.34 129.54 0)
+		(at 179.832 129.54 0)
 		(effects
 			(font
@@
 	(text "GND"
 		(exclude_from_sim no)
-		(at 180.34 127 0)
+		(at 179.832 127 0)
 		(effects
 			(font
@@
 	(text "SOA [MOSI]"
 		(exclude_from_sim no)
-		(at 184.15 121.92 0)
+		(at 183.388 121.92 0)
 		(effects
 			(font
@@
 	)
 	(junction
+		(at 165.1 78.74)
+		(diameter 0)
+		(color 0 0 0 0)
+	)
+	(junction
 		(at 55.88 73.66)
 		(diameter 0)
@@
 	)
 	(junction
-		(at 168.91 88.9)
-		(diameter 0)
-		(color 0 0 0 0)
-	)
-	(junction
 		(at 110.49 66.04)
 		(diameter 0)
@@
 	(wire
 		(pts
-			(xy 168.91 88.9) (xy 190.5 88.9)
+			(xy 151.13 33.02) (xy 151.13 86.36)
 		)
 		(stroke
@@
 	(wire
 		(pts
+			(xy 151.13 86.36) (xy 130.81 86.36)
+		)
+		(stroke
+			(width 0)
+			(type default)
+		)
+	)
+	(wire
+		(pts
 			(xy 113.03 68.58) (xy 113.03 66.04)
 		)
@@
 	(wire
 		(pts
-			(xy 130.81 81.28) (xy 151.13 81.28)
-		)
-		(stroke
-			(width 0)
-			(type default)
-		)
-	)
-	(wire
-		(pts
 			(xy 130.81 106.68) (xy 140.97 106.68)
 		)
@@
 	(wire
 		(pts
+			(xy 156.21 39.37) (xy 156.21 81.28)
+		)
+		(stroke
+			(width 0)
+			(type default)
+		)
+	)
+	(wire
+		(pts
 			(xy 199.39 39.37) (xy 199.39 41.91)
 		)
@@
 	(wire
 		(pts
-			(xy 156.21 39.37) (xy 156.21 86.36)
-		)
-		(stroke
-			(width 0)
-			(type default)
-		)
-	)
-	(wire
-		(pts
 			(xy 91.44 29.21) (xy 104.14 29.21)
 		)
@@
 	(wire
 		(pts
+			(xy 156.21 81.28) (xy 130.81 81.28)
+		)
+		(stroke
+			(width 0)
+			(type default)
+		)
+	)
+	(wire
+		(pts
 			(xy 130.81 99.06) (xy 133.35 99.06)
 		)
@@
 	(wire
 		(pts
-			(xy 168.91 82.55) (xy 168.91 88.9)
+			(xy 165.1 73.66) (xy 165.1 78.74)
 		)
 		(stroke
@@
 	(wire
 		(pts
+			(xy 165.1 78.74) (xy 165.1 88.9)
+		)
+		(stroke
+			(width 0)
+			(type default)
+		)
+	)
+	(wire
+		(pts
 			(xy 200.66 102.87) (xy 200.66 105.41)
 		)
@@
 	(wire
 		(pts
-			(xy 165.1 88.9) (xy 168.91 88.9)
+			(xy 165.1 88.9) (xy 190.5 88.9)
 		)
 		(stroke
@@
 	(wire
 		(pts
-			(xy 130.81 86.36) (xy 156.21 86.36)
-		)
-		(stroke
-			(width 0)
-			(type default)
-		)
-	)
-	(wire
-		(pts
 			(xy 104.14 43.18) (xy 104.14 45.72)
 		)
@@
 	(wire
 		(pts
-			(xy 151.13 33.02) (xy 151.13 81.28)
-		)
-		(stroke
-			(width 0)
-			(type default)
-		)
-	)
-	(wire
-		(pts
 			(xy 110.49 149.86) (xy 110.49 154.94)
 		)
@@
 		(pts
 			(xy 55.88 57.15) (xy 55.88 60.96)
-		)
-		(stroke
-			(width 0)
-			(type default)
-		)
-	)
-	(wire
-		(pts
-			(xy 165.1 78.74) (xy 165.1 88.9)
 		)
 		(stroke
@@
 	)
 	(label "IO0"
-		(at 168.91 82.55 0)
+		(at 165.1 73.66 0)
 		(effects
 			(font

Commit message: init
Parts:
- added Q1, Q2: BCW66G, Package_TO_SOT_SMD:SOT-23, symbol Simulation_SPICE:NPN
- added R6, R7: 10K, Resistor_SMD:R_1206_3216Metric, symbol Device:R
- added R8, R9: 470, Resistor_SMD:R_1206_3216Metric, symbol Device:R
- added U2: CH340C, Package_SO:SOIC-16_3.9x9.9mm_P1.27mm, symbol Interface_USB:CH340C
- D1: value LED -> green
- D2: value LED -> blue
- renumbered R5 to R4, R4 to R5
Connections:
- net +3.3V: now also U2.16 (VCC), U2.4 (V3)
- net CTS: now also U2.9 (~{CTS})
- net EN: now also Q1.1 (C)
- net GND: now also U2.1 (GND)
- net IO0: now also Q2.1 (C)
- net RTS: now also Q1.3 (E), R7.1, U2.14 (~{RTS})
- net at J1.4 (Pin_4): now also U1.33 (IO8); no longer U1.36 (IO23)
- net at J1.5 (Pin_5): now also U1.32 (SD0/IO7); no longer U1.35 (IO18)
- net supply/RXD renamed TXD0
- net TXD0: now also R9.2
- net supply/TXD renamed RXD0
- net RXD0: now also R8.2
- new net: R8.1, U2.2 (TXD)
- new net: R9.1, U2.3 (RXD)
- new net: Q2.2 (B), R7.2
- new net: Q1.2 (B), R6.2
- new net DTR: Q2.3 (E), R6.1, U2.13 (~{DTR})
- new net Supply_2/D+: U2.5 (UD+)
- new net Supply_2/D-: U2.6 (UD-)
- no-connect marks 24 -> 25
Other:
- removed sheet supply
- added sheet Supply_2 (supply_2.kicad_sch)
- moved on the sheet: C1, C2, C3, C4, D1, D2, J1, L1, R1, R2, R3, R4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
